Commit message: improved collision model

File: navi_model/urdf/gps.urdf.xacro (robot description, xacro)
@@ -9,4 +9,6 @@
     <xacro:property name="gps_x" value="-0.18941"/>
     <xacro:property name="gps_z" value="0.76387"/>
+    <xacro:property name="gps_rate" value="2.000"/>
+    <xacro:property name="gps_sigma" value="0.015"/>
     <xacro:macro name="gps">
         <joint name="gps_joint" type="fixed">
@@ -21,16 +23,14 @@
         </link>
         <gazebo>
-            <canonicalBody>gps_link</canonicalBody>
             <controller:gazebo_ros_p3d name="gps_controller" plugin="libgazebo_ros_p3d.so">
                 <alwaysOn>true</alwaysOn>
-                <updateRate>0.5</updateRate>
-                <bodyName>gps_link</bodyName>
-                <topicName>gps</topicName>
-                <gaussianNoise>${gps_noise}</gaussianNoise>
+                <updateRate>${gps_rate}</updateRate>
+                <bodyName>base_link</bodyName>
+                <topicName>/gps</topicName>
+                <gaussianNoise>${gps_sigma}</gaussianNoise>
                 <frameName>/map</frameName>
-                <xyzOffsets>0 0 0</xyzOffsets>
-                <rpyOffsets>0 0 0</rpyOffsets>
                 <interface:position name="gps_iface"/>
             </controller:gazebo_ros_p3d>
+            <canonicalBody>base_link</canonicalBody>
         </gazebo>
     </xacro:macro>

File: navi_model/urdf/navi.urdf.xacro (robot description, xacro)
@@ -18,8 +18,4 @@
         </inertial>
     </xacro:macro>
-    <xacro:property name="robot_width"  value="0.850"/>
-    <xacro:property name="robot_length" value="1.350"/>
-    <xacro:property name="robot_height" value="1.000"/>
-    <xacro:property name="robot_weight" value="20"/>
     <xacro:property name="caster_radius" value="0.102"/>
     <xacro:property name="caster_width"  value="0.075"/>

File: navi_model/urdf/navi_robot.urdf.xacro (robot description, xacro)
@@ -7,6 +7,9 @@
        xmlns:sensor="http://playerstage.sourceforge.net/gazebo/xmlschema/#sensor"
        xmlns:xacro="http://ros.org/wiki/xacro">
+    <xacro:property name="robot_width"  value="0.850"/>
+    <xacro:property name="robot_length" value="1.350"/>
+    <xacro:property name="robot_height" value="0.100"/>
+    <xacro:property name="robot_weight" value="20"/>
     <xacro:property name="offset_width"  value="0.600"/>
-    <xacro:property name="offset_height" value="0.000"/>
     <xacro:property name="offset_length" value="0.600"/>
     <link name="base_link">
@@ -19,11 +22,11 @@
         <!-- TODO: This bounding box isn't very accurate. -->
         <collision>
-            <origin xyz="0 0 ${robot_height/2+wheel_radius}" rpy="0 0 0"/>
+            <origin xyz="-0.25 0 ${2*wheel_radius}" rpy="0 0 0"/>
             <geometry>
-                <box size="${robot_length/2} ${robot_width} ${robot_height-wheel_radius}"/>
+                <box size="0.83 0.60 0.25"/>
             </geometry>
         </collision>
         <visual>
-            <origin xyz="-${offset_length} ${offset_width/2} -${offset_height}" rpy="${PI/2} 0 0"/>
+            <origin xyz="-0.6 0.3 0.0" rpy="${PI/2} 0 0"/>
             <geometry>
                 <mesh filename="package://navi_model/meshes/frame.stl" scale="0.001 0.001 0.001"/>
