Commit message: relative to base_link

File: navi_model/urdf/caster.urdf.xacro (robot description, xacro)
@@ -7,9 +7,12 @@
        xmlns:sensor="http://playerstage.sourceforge.net/gazebo/xmlschema/#sensor"
        xmlns:xacro="http://ros.org/wiki/xacro">
+    <xacro:property name="caster_offset_length" value="0.53388"/>
+    <xacro:property name="caster_offset_height" value="0.10833"/>
+    <xacro:property name="caster_trail_height"  value="0.00250"/>
     <xacro:macro name="caster">
         <joint name="caster_pivot_joint" type="continuous">
-            <parent link="base_footprint"/>
+            <parent link="base_link"/>
             <child link="caster_pivot_link"/>
-            <origin xyz="${-caster_offset} 0 ${2*caster_radius}" rpy="0 0 0"/>
+            <origin xyz="${-caster_offset_length} 0 ${caster_offset_height}" rpy="0 0 0"/>
             <axis xyz="0 0 1"/>
             <anchor xyz="0 0 0"/>
@@ -22,4 +25,11 @@
                                                  izz="0.001"/>
             </inertial>
+            <visual>
+                <origin xyz="0 0 0" rpy="0 0 0"/>
+                <geometry>
+                    <cylinder radius="0.05" length="0.025"/>
+                </geometry>
+                <material name="red"/>
+            </visual>
         </link>
         <gazebo reference="caster_pivot_link">
@@ -29,5 +39,5 @@
             <parent link="caster_pivot_link"/>
             <child link="caster_link"/>
-            <origin xyz="${-caster_trail} 0 ${-caster_radius}" rpy="0 0 0"/>
+            <origin xyz="${-caster_trail} 0 ${-caster_trail_height}" rpy="0 0 0"/>
             <axis xyz="0 1 0"/>
             <anchor xyz="0 0 0"/>
@@ -37,15 +47,15 @@
                 <mass value="${caster_weight}"/>
                 <inertia ixx="01" ixy="0.000" ixz="0.000"
-                                     iyy="0.1" iyz="0.000"
-                                                 izz="0.1"/>
+                                  iyy="0.100" iyz="0.000"
+                                              izz="0.100"/>
             </inertial>
             <collision>
                 <origin xyz="0 0 0" rpy="${PI/2} 0 0"/>
                 <geometry>
-                    <cylinder radius="${caster_radius}" length="${caster_width}"/>
+                    <mesh filename="package://navi_model/meshes/caster.stl" scale="0.001 0.001 0.001"/>
                 </geometry>
             </collision>
             <visual>
-                <origin xyz="0 0 0" rpy="${PI/2} 0 0"/>
+                <origin xyz="0 0 -${caster_radius}" rpy="${PI/2} 0 0"/>
                 <geometry>
                     <cylinder radius="${caster_radius}" length="${caster_width}"/>

File: navi_model/urdf/navi.urdf.xacro (robot description, xacro)
@@ -13,5 +13,4 @@
     <xacro:property name="robot_height" value="1.000"/>
     <xacro:property name="robot_weight" value="20"/>
-    <xacro:property name="robot_radius" value="0.70354"/>
     <xacro:property name="caster_radius" value="0.102"/>
     <xacro:property name="caster_width"  value="0.075"/>
@@ -24,13 +23,13 @@
     <include filename="$(find navi_model)/urdf/navi_robot.urdf.xacro"/>
     <include filename="$(find navi_model)/urdf/wheels.urdf.xacro"/>
+    <include filename="$(find navi_model)/urdf/caster.urdf.xacro"/>
     <!--
-    <include filename="$(find navi_model)/urdf/caster.urdf.xacro"/>
     <include filename="$(find navi_model)/urdf/sensors.urdf.xacro"/>
     -->
     <xacro:wheel side="left"  sign="+1"/>
     <xacro:wheel side="right" sign="-1"/>
-    <!--
     <xacro:caster/>
     <xacro:driver/>
+    <!--
     <xacro:gps/>
     -->

File: navi_model/urdf/navi_robot.urdf.xacro (robot description, xacro)
@@ -8,5 +8,5 @@
        xmlns:xacro="http://ros.org/wiki/xacro">
     <xacro:property name="offset_width"  value="0.600"/>
-    <xacro:property name="offset_height" value="0.07"/>
+    <xacro:property name="offset_height" value="0.000"/>
     <xacro:property name="offset_length" value="0.600"/>
     <link name="base_link">
@@ -35,3 +35,11 @@
         <material>Gazebo/Blue</material>
     </gazebo>
+    <joint name="base_footprint_joint" type="fixed">
+        <parent link="base_link"/>
+        <child link="base_footprint"/>
+        <origin xyz="0 0 ${-wheel_radius}" rpy="0 0 0"/>
+        <axis xyz="0 0 0"/>
+        <anchor xyz="0 0 0"/>
+    </joint>
+    <link name="base_footprint"/>
 </robot>

Commit message: switched to caster model

File: navi_model/urdf/caster.urdf.xacro (robot description, xacro)
@@ -9,5 +9,6 @@
     <xacro:property name="caster_offset_length" value="0.53388"/>
     <xacro:property name="caster_offset_height" value="0.10833"/>
-    <xacro:property name="caster_trail_height"  value="0.00250"/>
+    <xacro:property name="caster_trail_height"  value="0.12000"/>
+    <xacro:property name="caster_width" value="0.1"/>
     <xacro:macro name="caster">
         <joint name="caster_pivot_joint" type="continuous">
@@ -25,11 +26,4 @@
                                                  izz="0.001"/>
             </inertial>
-            <visual>
-                <origin xyz="0 0 0" rpy="0 0 0"/>
-                <geometry>
-                    <cylinder radius="0.05" length="0.025"/>
-                </geometry>
-                <material name="red"/>
-            </visual>
         </link>
         <gazebo reference="caster_pivot_link">
@@ -53,11 +47,11 @@
                 <origin xyz="0 0 0" rpy="${PI/2} 0 0"/>
                 <geometry>
-                    <mesh filename="package://navi_model/meshes/caster.stl" scale="0.001 0.001 0.001"/>
+                    <cylinder radius="${caster_radius}" length="${caster_width}"/>
                 </geometry>
             </collision>
             <visual>
-                <origin xyz="0 0 -${caster_radius}" rpy="${PI/2} 0 0"/>
+                <origin xyz="${caster_radius} ${-caster_width/2} ${-caster_radius}" rpy="${PI/2} 0 ${PI}"/>
                 <geometry>
-                    <cylinder radius="${caster_radius}" length="${caster_width}"/>
+                    <mesh filename="package://navi_model/meshes/caster.stl" scale="0.001 0.001 0.001"/>
                 </geometry>
                 <material name="red"/>

Commit message: fixed height in spawn script

File: navi_model/urdf/caster.urdf.xacro (robot description, xacro)
@@ -20,10 +20,5 @@
         </joint>
         <link name="caster_pivot_link">
-            <inertial>
-                <mass value="0.001"/>
-                <inertia ixx="0.001" ixy="0.000" ixz="0.000"
-                                     iyy="0.001" iyz="0.000"
-                                                 izz="0.001"/>
-            </inertial>
+            <xacro:weightless/>
         </link>
         <gazebo reference="caster_pivot_link">
@@ -40,7 +35,7 @@
             <inertial>
                 <mass value="${caster_weight}"/>
-                <inertia ixx="01" ixy="0.000" ixz="0.000"
-                                  iyy="0.100" iyz="0.000"
-                                              izz="0.100"/>
+                <inertia ixx="0.100" ixy="0.000" ixz="0.000"
+                                     iyy="0.100" iyz="0.000"
+                                                 izz="0.100"/>
             </inertial>
             <collision>

Commit message: fixed the caster's animation

File: navi_model/urdf/caster.urdf.xacro (robot description, xacro)
@@ -9,6 +9,10 @@
     <xacro:property name="caster_offset_length" value="0.53388"/>
     <xacro:property name="caster_offset_height" value="0.10833"/>
-    <xacro:property name="caster_trail_height"  value="0.12000"/>
-    <xacro:property name="caster_width" value="0.1"/>
+    <xacro:property name="caster_trail_height" value="0.12000"/>
+    <xacro:property name="caster_trail_length" value="0.01"/>
+    <xacro:property name="caster_radius" value="0.102"/>
+    <xacro:property name="caster_width"  value="0.075"/>
+    <xacro:property name="caster_weight" value="1.225"/>
+    <xacro:property name="caster_width" value="0.06"/>
     <xacro:macro name="caster">
         <joint name="caster_pivot_joint" type="continuous">
@@ -20,4 +24,12 @@
         </joint>
         <link name="caster_pivot_link">
+            <visual>
+                <origin xyz="${caster_radius} -0.055 ${-caster_radius - caster_trail_height}"
+                        rpy="${PI/2} 0 ${PI}"/>
+                <geometry>
+                    <mesh filename="package://navi_model/meshes/caster.stl" scale="0.001 0.001 0.001"/>
+                </geometry>
+                <material name="red"/>
+            </visual>
             <xacro:weightless/>
         </link>
@@ -28,5 +40,5 @@
             <parent link="caster_pivot_link"/>
             <child link="caster_link"/>
-            <origin xyz="${-caster_trail} 0 ${-caster_trail_height}" rpy="0 0 0"/>
+            <origin xyz="${-caster_trail_length} 0 ${-caster_trail_height}" rpy="0 0 0"/>
             <axis xyz="0 1 0"/>
             <anchor xyz="0 0 0"/>
@@ -45,11 +57,4 @@
                 </geometry>
             </collision>
-            <visual>
-                <origin xyz="${caster_radius} ${-caster_width/2} ${-caster_radius}" rpy="${PI/2} 0 ${PI}"/>
-                <geometry>
-                    <mesh filename="package://navi_model/meshes/caster.stl" scale="0.001 0.001 0.001"/>
-                </geometry>
-                <material name="red"/>
-            </visual>
         </link>
         <gazebo reference="caster_link">

File: navi_model/urdf/navi.urdf.xacro (robot description, xacro)
@@ -18,9 +18,4 @@
         </inertial>
     </xacro:macro>
-    <xacro:property name="caster_radius" value="0.102"/>
-    <xacro:property name="caster_width"  value="0.075"/>
-    <xacro:property name="caster_offset" value="0.500"/>
-    <xacro:property name="caster_trail"  value="0.050"/>
-    <xacro:property name="caster_weight" value="1.225"/>
     <xacro:property name="gps_noise" value="0.005"/>
     <xacro:property name="encoders_noise" value="0.100"/>

File: navi_model/urdf/navi_robot.urdf.xacro (robot description, xacro)
@@ -11,6 +11,4 @@
     <xacro:property name="robot_height" value="0.100"/>
     <xacro:property name="robot_weight" value="20"/>
-    <xacro:property name="offset_width"  value="0.600"/>
-    <xacro:property name="offset_length" value="0.600"/>
     <link name="base_link">
         <inertial>

Commit message: works, but the caster is too laggy

File: navi_model/urdf/caster.urdf.xacro (robot description, xacro)
@@ -21,5 +21,4 @@
             <origin xyz="${-caster_offset_length} 0 ${caster_offset_height}" rpy="0 0 0"/>
             <axis xyz="0 0 1"/>
-            <anchor xyz="0 0 0"/>
         </joint>
         <link name="caster_pivot_link">
@@ -32,5 +31,16 @@
                 <material name="red"/>
             </visual>
-            <xacro:weightless/>
+            <collision>
+                <origin xyz="0 0 0" rpy="0 0 0"/>
+                <geometry>
+                    <box size="${EPS} ${EPS} ${EPS}"/>
+                </geometry>
+            </collision>
+            <inertial>
+                <mass value="0.01"/>
+                <inertia ixx="0.01" ixy="0.000"  ixz="0.000"
+                                     iyy="0.01" iyz="0.000"
+                                                  izz="0.01"/>
+            </inertial>
         </link>
         <gazebo reference="caster_pivot_link">
@@ -42,5 +52,4 @@
             <origin xyz="${-caster_trail_length} 0 ${-caster_trail_height}" rpy="0 0 0"/>
             <axis xyz="0 1 0"/>
-            <anchor xyz="0 0 0"/>
         </joint>
         <link name="caster_link">
@@ -57,4 +66,11 @@
                 </geometry>
             </collision>
+            <visual>
+                <origin xyz="0 0 0" rpy="${PI/2} 0 0"/>
+                <geometry>
+                    <cylinder radius="${caster_radius}" length="${caster_width}"/>
+                </geometry>
+                <material name="red"/>
+            </visual>
         </link>
         <gazebo reference="caster_link">

Commit message: fixed caster inertia

File: navi_model/urdf/caster.urdf.xacro (robot description, xacro)
@@ -38,8 +38,8 @@
             </collision>
             <inertial>
-                <mass value="0.01"/>
-                <inertia ixx="0.01" ixy="0.000"  ixz="0.000"
-                                     iyy="0.01" iyz="0.000"
-                                                  izz="0.01"/>
+                <mass value="0.1"/>
+                <inertia ixx="0.01241" ixy="0.0"     ixz="0.00000"
+                                       iyy="0.01522" iyz="0.00000"
+                                                     izz="0.01176"/>
             </inertial>
         </link>
@@ -55,8 +55,8 @@
         <link name="caster_link">
             <inertial>
-                <mass value="${caster_weight}"/>
-                <inertia ixx="0.100" ixy="0.000" ixz="0.000"
-                                     iyy="0.100" iyz="0.000"
-                                                 izz="0.100"/>
+                <mass value="0.1"/>
+                <inertia ixx="0.01241" ixy="0.0"     ixz="0.00000"
+                                       iyy="0.01522" iyz="0.00000"
+                                                     izz="0.01176"/>
             </inertial>
             <collision>

Commit message: caster weighs too much, but closer

File: navi_model/urdf/caster.urdf.xacro (robot description, xacro)
@@ -10,5 +10,5 @@
     <xacro:property name="caster_offset_height" value="0.10833"/>
     <xacro:property name="caster_trail_height" value="0.12000"/>
-    <xacro:property name="caster_trail_length" value="0.01"/>
+    <xacro:property name="caster_trail_length" value="0.1"/>
     <xacro:property name="caster_radius" value="0.102"/>
     <xacro:property name="caster_width"  value="0.075"/>

File: navi_model/urdf/navi_robot.urdf.xacro (robot description, xacro)
@@ -10,11 +10,12 @@
     <xacro:property name="robot_length" value="1.350"/>
     <xacro:property name="robot_height" value="0.100"/>
-    <xacro:property name="robot_weight" value="20"/>
+    <xacro:property name="robot_weight" value="90.718"/>
     <link name="base_link">
         <inertial>
+            <origin xyz="-0.4 0.0 0.3" rpy="0 0 0"/>
             <mass value="${robot_weight}"/>
-            <inertia ixx="1.000" ixy="0.000" ixz="0.000"
-                                 iyy="1.000" iyz="0.000"
-                                             izz="1.000"/>
+            <inertia ixx="1.000" ixy="0.000"  ixz="0.000"
+                                 iyy="28.500" iyz="0.000"
+                                              izz="34.800"/>
         </inertial>
         <!-- TODO: This bounding box isn't very accurate. -->

Commit message: caster sorta works

File: navi_model/urdf/caster.urdf.xacro (robot description, xacro)
@@ -10,5 +10,5 @@
     <xacro:property name="caster_offset_height" value="0.10833"/>
     <xacro:property name="caster_trail_height" value="0.12000"/>
-    <xacro:property name="caster_trail_length" value="0.1"/>
+    <xacro:property name="caster_trail_length" value="0.05"/>
     <xacro:property name="caster_radius" value="0.102"/>
     <xacro:property name="caster_width"  value="0.075"/>
@@ -38,5 +38,5 @@
             </collision>
             <inertial>
-                <mass value="0.1"/>
+                <mass value="0.05"/>
                 <inertia ixx="0.01241" ixy="0.0"     ixz="0.00000"
                                        iyy="0.01522" iyz="0.00000"
@@ -55,5 +55,5 @@
         <link name="caster_link">
             <inertial>
-                <mass value="0.1"/>
+                <mass value="0.05"/>
                 <inertia ixx="0.01241" ixy="0.0"     ixz="0.00000"
                                        iyy="0.01522" iyz="0.00000"
