Commit message: Moved base_link and switched to new model.

File: navi_model/urdf/navi.urdf.xacro (robot description, xacro)
@@ -26,4 +26,5 @@
     <include filename="$(find navi_model)/urdf/materials.urdf.xacro"/>
     <include filename="$(find navi_model)/urdf/navi_robot.urdf.xacro"/>
+    <!--
     <include filename="$(find navi_model)/urdf/wheels.urdf.xacro"/>
     <include filename="$(find navi_model)/urdf/caster.urdf.xacro"/>
@@ -34,3 +35,4 @@
     <xacro:driver/>
     <xacro:gps/>
+    -->
 </robot>

File: navi_model/urdf/navi_robot.urdf.xacro (robot description, xacro)
@@ -7,5 +7,8 @@
        xmlns:sensor="http://playerstage.sourceforge.net/gazebo/xmlschema/#sensor"
        xmlns:xacro="http://ros.org/wiki/xacro">
-    <link name="base_footprint">
+    <xacro:property name="offset_width"  value="0.600"/>
+    <xacro:property name="offset_height" value="0.127"/>
+    <xacro:property name="offset_length" value="0.600"/>
+    <link name="base_link">
         <inertial>
             <mass value="${robot_weight}"/>
@@ -22,12 +25,12 @@
         </collision>
         <visual>
-            <origin xyz="${-robot_length/2} ${robot_width/2} 0" rpy="${PI/2} 0 0"/>
+            <origin xyz="-${offset_length} ${offset_width/2} -${offset_height}" rpy="${PI/2} 0 0"/>
             <geometry>
-                <mesh filename="package://navi_model/meshes/navi2.stl" scale="0.001 0.001 0.001"/>
+                <mesh filename="package://navi_model/meshes/frame.stl" scale="0.001 0.001 0.001"/>
             </geometry>
             <material name="blue"/>
         </visual>
     </link>
-    <gazebo reference="base_footprint">
+    <gazebo reference="base_link">
         <material>Gazebo/Blue</material>
     </gazebo>

Commit message: moved wheels to the correct location

File: navi_model/urdf/navi.urdf.xacro (robot description, xacro)
@@ -13,8 +13,5 @@
     <xacro:property name="robot_height" value="1.000"/>
     <xacro:property name="robot_weight" value="20"/>
-    <xacro:property name="wheel_radius" value="0.127"/>
-    <xacro:property name="wheel_width"  value="0.100"/>
-    <xacro:property name="wheel_offset" value="0.425"/>
-    <xacro:property name="wheel_weight" value="1.687"/>
+    <xacro:property name="robot_radius" value="0.70354"/>
     <xacro:property name="caster_radius" value="0.102"/>
     <xacro:property name="caster_width"  value="0.075"/>
@@ -26,10 +23,12 @@
     <include filename="$(find navi_model)/urdf/materials.urdf.xacro"/>
     <include filename="$(find navi_model)/urdf/navi_robot.urdf.xacro"/>
+    <include filename="$(find navi_model)/urdf/wheels.urdf.xacro"/>
     <!--
-    <include filename="$(find navi_model)/urdf/wheels.urdf.xacro"/>
     <include filename="$(find navi_model)/urdf/caster.urdf.xacro"/>
     <include filename="$(find navi_model)/urdf/sensors.urdf.xacro"/>
+    -->
     <xacro:wheel side="left"  sign="+1"/>
     <xacro:wheel side="right" sign="-1"/>
+    <!--
     <xacro:caster/>
     <xacro:driver/>

File: navi_model/urdf/navi_robot.urdf.xacro (robot description, xacro)
@@ -8,5 +8,5 @@
        xmlns:xacro="http://ros.org/wiki/xacro">
     <xacro:property name="offset_width"  value="0.600"/>
-    <xacro:property name="offset_height" value="0.127"/>
+    <xacro:property name="offset_height" value="0.07"/>
     <xacro:property name="offset_length" value="0.600"/>
     <link name="base_link">

File: navi_model/urdf/wheels.urdf.xacro (robot description, xacro)
@@ -7,9 +7,13 @@
        xmlns:sensor="http://playerstage.sourceforge.net/gazebo/xmlschema/#sensor"
        xmlns:xacro="http://ros.org/wiki/xacro">
+    <xacro:property name="wheel_radius" value="0.127"/>
+    <xacro:property name="wheel_width"  value="0.100"/>
+    <xacro:property name="wheel_offset" value="0.35193"/>
+    <xacro:property name="wheel_weight" value="1.687"/>
     <xacro:macro name="wheel" params="side sign">
         <joint name="wheel_${side}_joint" type="continuous">
-            <parent link="base_footprint"/>
+            <parent link="base_link"/>
             <child link="wheel_${side}_link"/>
-            <origin xyz="0 ${sign*wheel_offset} ${wheel_radius}"/>
+            <origin xyz="0 ${sign*wheel_offset} 0"/>
             <axis xyz="0 1 0"/>
             <anchor xyz="0 0 0"/>

Commit message: added laser to simulation

File: navi_model/urdf/navi.urdf.xacro (robot description, xacro)
@@ -24,13 +24,10 @@
     <include filename="$(find navi_model)/urdf/wheels.urdf.xacro"/>
     <include filename="$(find navi_model)/urdf/caster.urdf.xacro"/>
-    <!--
     <include filename="$(find navi_model)/urdf/sensors.urdf.xacro"/>
-    -->
     <xacro:wheel side="left"  sign="+1"/>
     <xacro:wheel side="right" sign="-1"/>
     <xacro:caster/>
     <xacro:driver/>
-    <!--
+    <xacro:laser/>
     <xacro:gps/>
-    -->
 </robot>

File: navi_model/urdf/sensors.urdf.xacro (robot description, xacro)
@@ -7,4 +7,67 @@
        xmlns:sensor="http://playerstage.sourceforge.net/gazebo/xmlschema/#sensor"
        xmlns:xacro="http://ros.org/wiki/xacro">
+    <xacro:property name="gps_x" value="-0.18941"/>
+    <xacro:property name="gps_z" value="0.76387"/>
+    <xacro:property name="laser_x" value="0.02927"/>
+    <xacro:property name="laser_z" value="0.46714"/>
+    <!-- GPS -->
+    <xacro:macro name="gps">
+        <joint name="gps_joint" type="fixed">
+            <parent link="base_link"/>
+            <child link="gps_link"/>
+            <origin xyz="${gps_x} 0 ${gps_z}" rpy="0 0 0"/>
+            <axis xyz="0 0 0"/>
+            <anchor xyz="0 0 0"/>
+        </joint>
+        <link name="gps_link"/>
+        <gazebo>
+            <canonicalBody>gps_link</canonicalBody>
+            <controller:gazebo_ros_p3d name="gps_controller" plugin="libgazebo_ros_p3d.so">
+                <alwaysOn>true</alwaysOn>
+                <updateRate>0.5</updateRate>
+                <bodyName>gps_link</bodyName>
+                <topicName>gps</topicName>
+                <gaussianNoise>${gps_noise}</gaussianNoise>
+                <frameName>/map</frameName>
+                <xyzOffsets>0 0 0</xyzOffsets>
+                <rpyOffsets>0 0 0</rpyOffsets>
+                <interface:position name="gps_iface"/>
+            </controller:gazebo_ros_p3d>
+        </gazebo>
+    </xacro:macro>
+    <!-- Laser -->
+    <xacro:macro name="laser">
+        <joint name="laser_joint" type="fixed">
+            <parent link="base_link"/>
+            <child link="laser_link"/>
+            <origin xyz="${laser_x} 0 ${laser_z}" rpy="0 0 0"/>
+            <axis xyz="0 0 0"/>
+            <anchor xyz="0 0 0"/>
+        </joint>
+        <link name="laser_link"/>
+        <gazebo reference="base_laser_link">
+            <sensor:ray name="laser">
+                <rayCount>640</rayCount>
+                <rangeCount>640</rangeCount>
+                <laserCount>1</laserCount>
+                <origin>0.0 0.0 0.0</origin>
+                <displayRays>false</displayRays>
+                <minAngle>-120</minAngle>
+                <maxAngle>120</maxAngle>
+                <minRange>0.08</minRange>
+                <maxRange>15.0</maxRange>
+                <resRange>0.01</resRange>
+                <updateRate>20</updateRate>
+                <controller:gazebo_ros_laser name="gazebo_ros_laser_controller" plugin="libgazebo_ros_laser.so">
+                    <gaussianNoise>0.005</gaussianNoise>
+                    <alwaysOn>true</alwaysOn>
+                    <updateRate>20</updateRate>
+                    <topicName>base_laser/scan</topicName>
+                    <frameName>base_laser_link</frameName>
+                    <interface:laser name="gazebo_ros_laser_iface"/>
+                </controller:gazebo_ros_laser>
+            </sensor:ray>
+        </gazebo>
+    </xacro:macro>
     <xacro:macro name="driver">
         <gazebo>
@@ -35,19 +98,3 @@
         </gazebo>
     </xacro:macro>
-    <xacro:macro name="gps">
-        <gazebo>
-            <canonicalBody>base_footprint</canonicalBody>
-            <controller:gazebo_ros_p3d name="gps_controller" plugin="libgazebo_ros_p3d.so">
-                <alwaysOn>true</alwaysOn>
-                <updateRate>0.5</updateRate>
-                <bodyName>base_footprint</bodyName>
-                <topicName>gps</topicName>
-                <gaussianNoise>${gps_noise}</gaussianNoise>
-                <frameName>/map</frameName>
-                <xyzOffsets>0 0 0</xyzOffsets>
-                <rpyOffsets>0 0 0</rpyOffsets>
-                <interface:position name="gps_iface"/>
-            </controller:gazebo_ros_p3d>
-        </gazebo>
-    </xacro:macro>
 </robot>

Commit message: split sensors into separate files

File: navi_model/urdf/navi.urdf.xacro (robot description, xacro)
@@ -25,4 +25,6 @@
     <include filename="$(find navi_model)/urdf/caster.urdf.xacro"/>
     <include filename="$(find navi_model)/urdf/sensors.urdf.xacro"/>
+    <include filename="$(find navi_model)/urdf/laser.urdf.xacro"/>
+    <include filename="$(find navi_model)/urdf/gps.urdf.xacro"/>
     <xacro:wheel side="left"  sign="+1"/>
     <xacro:wheel side="right" sign="-1"/>

File: navi_model/urdf/sensors.urdf.xacro (robot description, xacro)
@@ -7,67 +7,4 @@
        xmlns:sensor="http://playerstage.sourceforge.net/gazebo/xmlschema/#sensor"
        xmlns:xacro="http://ros.org/wiki/xacro">
-    <xacro:property name="gps_x" value="-0.18941"/>
-    <xacro:property name="gps_z" value="0.76387"/>
-    <xacro:property name="laser_x" value="0.02927"/>
-    <xacro:property name="laser_z" value="0.46714"/>
-    <!-- GPS -->
-    <xacro:macro name="gps">
-        <joint name="gps_joint" type="fixed">
-            <parent link="base_link"/>
-            <child link="gps_link"/>
-            <origin xyz="${gps_x} 0 ${gps_z}" rpy="0 0 0"/>
-            <axis xyz="0 0 0"/>
-            <anchor xyz="0 0 0"/>
-        </joint>
-        <link name="gps_link"/>
-        <gazebo>
-            <canonicalBody>gps_link</canonicalBody>
-            <controller:gazebo_ros_p3d name="gps_controller" plugin="libgazebo_ros_p3d.so">
-                <alwaysOn>true</alwaysOn>
-                <updateRate>0.5</updateRate>
-                <bodyName>gps_link</bodyName>
-                <topicName>gps</topicName>
-                <gaussianNoise>${gps_noise}</gaussianNoise>
-                <frameName>/map</frameName>
-                <xyzOffsets>0 0 0</xyzOffsets>
-                <rpyOffsets>0 0 0</rpyOffsets>
-                <interface:position name="gps_iface"/>
-            </controller:gazebo_ros_p3d>
-        </gazebo>
-    </xacro:macro>
-    <!-- Laser -->
-    <xacro:macro name="laser">
-        <joint name="laser_joint" type="fixed">
-            <parent link="base_link"/>
-            <child link="laser_link"/>
-            <origin xyz="${laser_x} 0 ${laser_z}" rpy="0 0 0"/>
-            <axis xyz="0 0 0"/>
-            <anchor xyz="0 0 0"/>
-        </joint>
-        <link name="laser_link"/>
-        <gazebo reference="base_laser_link">
-            <sensor:ray name="laser">
-                <rayCount>640</rayCount>
-                <rangeCount>640</rangeCount>
-                <laserCount>1</laserCount>
-                <origin>0.0 0.0 0.0</origin>
-                <displayRays>false</displayRays>
-                <minAngle>-120</minAngle>
-                <maxAngle>120</maxAngle>
-                <minRange>0.08</minRange>
-                <maxRange>15.0</maxRange>
-                <resRange>0.01</resRange>
-                <updateRate>20</updateRate>
-                <controller:gazebo_ros_laser name="gazebo_ros_laser_controller" plugin="libgazebo_ros_laser.so">
-                    <gaussianNoise>0.005</gaussianNoise>
-                    <alwaysOn>true</alwaysOn>
-                    <updateRate>20</updateRate>
-                    <topicName>base_laser/scan</topicName>
-                    <frameName>base_laser_link</frameName>
-                    <interface:laser name="gazebo_ros_laser_iface"/>
-                </controller:gazebo_ros_laser>
-            </sensor:ray>
-        </gazebo>
-    </xacro:macro>
     <xacro:macro name="driver">
         <gazebo>

Commit message: renders properly, at least

File: navi_model/urdf/navi.urdf.xacro (robot description, xacro)
@@ -10,28 +10,5 @@
     <xacro:property name="EPS" value="0.000001"/>
     <xacro:property name="PI" value="3.1415926535897931"/>
-    <xacro:property name="robot_weight" value="90.0"/>
-    <xacro:property name="wheel_radius" value="0.127"/>
-    <xacro:macro name="weightless">
-        <inertial>
-            <mass value="${EPS}"/>
-            <inertia ixx="${EPS}" ixy="0.000"  ixz="0.000"
-                                  iyy="${EPS}" iyz="0.000"
-                                               izz="${EPS}"/>
-        </inertial>
-    </xacro:macro>
-    <include filename="$(find navi_model)/urdf/materials.urdf.xacro"/>
     <include filename="$(find navi_model)/urdf/navi_robot.urdf.xacro"/>
-    <include filename="$(find navi_model)/urdf/wheels.urdf.xacro"/>
-    <include filename="$(find navi_model)/urdf/caster.urdf.xacro"/>
-    <include filename="$(find navi_model)/urdf/cameras.urdf.xacro"/>
-    <include filename="$(find navi_model)/urdf/laser.urdf.xacro"/>
-    <include filename="$(find navi_model)/urdf/gps.urdf.xacro"/>
-    <xacro:wheel side="left"  sign="+1"/>
-    <xacro:wheel side="right" sign="-1"/>
-    <xacro:caster/>
-    <xacro:driver/>
-    <xacro:laser/>
-    <xacro:gps/>
-    <xacro:camera side="left"  sign="+1"/>
-    <xacro:camera side="right" sign="-1"/>
+    <chassis/>
 </robot>

File: navi_model/urdf/navi_robot.urdf.xacro (robot description, xacro)
@@ -7,68 +7,22 @@
        xmlns:sensor="http://playerstage.sourceforge.net/gazebo/xmlschema/#sensor"
        xmlns:xacro="http://ros.org/wiki/xacro">
-    <xacro:property name="robot_width"  value="0.850"/>
-    <xacro:property name="robot_length" value="1.350"/>
-    <xacro:property name="robot_height" value="0.100"/>
-    <xacro:property name="robot_weight" value="90.718"/>
-    <link name="base_link">
-        <inertial>
-            <origin xyz="-0.4 0.0 0.3" rpy="0 0 0"/>
-            <mass value="${robot_weight}"/>
-            <inertia ixx="1.000" ixy="0.000"  ixz="0.000"
-                                 iyy="28.500" iyz="0.000"
-                                              izz="34.800"/>
-        </inertial>
-        <!-- TODO: This bounding box isn't very accurate. -->
-        <collision>
-            <origin xyz="-0.25 0 ${2*wheel_radius}" rpy="0 0 0"/>
-            <geometry>
-                <box size="0.83 0.60 0.25"/>
-            </geometry>
-        </collision>
-        <visual>
-            <origin xyz="-0.6 0.3 0.0" rpy="${PI/2} 0 0"/>
-            <geometry>
-                <mesh filename="package://navi_model/meshes/frame.stl" scale="0.001 0.001 0.001"/>
-            </geometry>
-            <material name="blue"/>
-        </visual>
-    </link>
-    <gazebo reference="base_link">
-        <material>Gazebo/Blue</material>
-    </gazebo>
-    <joint name="base_footprint_joint" type="fixed">
-        <parent link="base_link"/>
-        <child link="base_footprint"/>
-        <origin xyz="0 0 ${-wheel_radius}" rpy="0 0 0"/>
-        <axis xyz="0 0 0"/>
-        <anchor xyz="0 0 0"/>
-    </joint>
-    <link name="base_footprint">
-        <xacro:weightless/>
-    </link>
-    <gazebo>
-        <controller:diffdrive_plugin name="differential_drive_controller" plugin="libdiffdrive_plugin.so">
-            <alwaysOn>true</alwaysOn>
-            <update>100</update>
-            <updateRate>100.0</updateRate>
-            <torque>1000</torque>
-            <wheelSeparation>${wheel_offset*2}</wheelSeparation>
-            <wheelDiameter>${wheel_radius*2}</wheelDiameter>
-            <robotNamespace>/</robotNamespace>
-            <topicName>drive/cmd_vel</topicName>
-            <leftJoint>wheel_left_joint</leftJoint>
-            <rightJoint>wheel_right_joint</rightJoint>
-            <interface:position name="drive_iface"/>
-        </controller:diffdrive_plugin>
-        <controller:gazebo_ros_p3d name="gps_controller" plugin="libgazebo_ros_p3d.so">
-            <alwaysOn>true</alwaysOn>
-            <updateRate>60</updateRate>
-            <bodyName>base_link</bodyName>
-            <topicName>ground_truth</topicName>
-            <gaussianNoise>0.0</gaussianNoise>
-            <frameName>/map</frameName>
-            <interface:position name="gps_iface"/>
-        </controller:gazebo_ros_p3d>
-        <canonicalBody>base_footprint</canonicalBody>
-    </gazebo>
+    <xacro:macro name="chassis">
+        <link name="base_link">
+            <collision name="collision">
+                <geometry><box size="1.5 1.0 0.2"/></geometry>
+            </collision>
+            <visual>
+                <origin xyz="-0.6 0.3 -0.127" rpy="${PI/2} 0 0"/>
+                <geometry>
+                    <mesh filename="package://navi_model/meshes/frame.stl" scale="0.001 0.001 0.001"/>
+                </geometry>
+            </visual>
+            <inertial>
+                <mass value="${EPS}"/>
+                <inertia ixx="${EPS}" ixy="0"      ixz="0"
+                                      iyy="${EPS}" iyz="0"
+                                                   izz="${EPS}"/>
+            </inertial>
+        </link>
+    </xacro:macro>
 </robot>

Commit message: Revert "renders properly, at least"
This reverts commit 44ae823b0eb2c91112526bfdef02392b4b58d1ff.

File: navi_model/urdf/navi.urdf.xacro (robot description, xacro)
@@ -10,5 +10,28 @@
     <xacro:property name="EPS" value="0.000001"/>
     <xacro:property name="PI" value="3.1415926535897931"/>
+    <xacro:property name="robot_weight" value="90.0"/>
+    <xacro:property name="wheel_radius" value="0.127"/>
+    <xacro:macro name="weightless">
+        <inertial>
+            <mass value="${EPS}"/>
+            <inertia ixx="${EPS}" ixy="0.000"  ixz="0.000"
+                                  iyy="${EPS}" iyz="0.000"
+                                               izz="${EPS}"/>
+        </inertial>
+    </xacro:macro>
+    <include filename="$(find navi_model)/urdf/materials.urdf.xacro"/>
     <include filename="$(find navi_model)/urdf/navi_robot.urdf.xacro"/>
-    <chassis/>
+    <include filename="$(find navi_model)/urdf/wheels.urdf.xacro"/>
+    <include filename="$(find navi_model)/urdf/caster.urdf.xacro"/>
+    <include filename="$(find navi_model)/urdf/cameras.urdf.xacro"/>
+    <include filename="$(find navi_model)/urdf/laser.urdf.xacro"/>
+    <include filename="$(find navi_model)/urdf/gps.urdf.xacro"/>
+    <xacro:wheel side="left"  sign="+1"/>
+    <xacro:wheel side="right" sign="-1"/>
+    <xacro:caster/>
+    <xacro:driver/>
+    <xacro:laser/>
+    <xacro:gps/>
+    <xacro:camera side="left"  sign="+1"/>
+    <xacro:camera side="right" sign="-1"/>
 </robot>
