Commit message: added caster parameters

File: navi_model/urdf/navi.urdf.xacro (robot description, xacro)
@@ -12,26 +12,106 @@
     <xacro:property name="robot_weight" value="90.0"/>
     <xacro:property name="wheel_radius" value="0.127"/>
-    <xacro:macro name="weightless">
+    <xacro:property name="wheel_thickness" value="0.05"/>
+    <link name="base_link">
         <inertial>
-            <mass value="${EPS}"/>
-            <inertia ixx="${EPS}" ixy="0.000"  ixz="0.000"
-                                  iyy="${EPS}" iyz="0.000"
-                                               izz="${EPS}"/>
+            <origin xyz="0 0 0"/>
+            <mass value="1.0"/>
+            <inertia ixx="1.0" ixy="0.0"   ixz="0.0"
+                               iyy="100.0" iyz="0.0"
+                                           izz="1.0" />
         </inertial>
-    </xacro:macro>
-    <include filename="$(find navi_model)/urdf/materials.urdf.xacro"/>
-    <include filename="$(find navi_model)/urdf/navi_robot.urdf.xacro"/>
-    <include filename="$(find navi_model)/urdf/wheels.urdf.xacro"/>
-    <include filename="$(find navi_model)/urdf/caster.urdf.xacro"/>
-    <include filename="$(find navi_model)/urdf/cameras.urdf.xacro"/>
-    <include filename="$(find navi_model)/urdf/laser.urdf.xacro"/>
-    <include filename="$(find navi_model)/urdf/gps.urdf.xacro"/>
-    <xacro:wheel side="left"  sign="+1"/>
-    <xacro:wheel side="right" sign="-1"/>
-    <xacro:caster/>
-    <xacro:driver/>
-    <xacro:laser/>
-    <xacro:gps/>
-    <xacro:camera side="left"  sign="+1"/>
-    <xacro:camera side="right" sign="-1"/>
+        <visual>
+            <origin xyz="0 0 0"/>
+            <geometry>
+                <box size="0.9 0.8 0.3"/>
+            </geometry>
+        </visual>
+        <collision>
+            <origin xyz="0 0 0"/>
+            <geometry>
+                <box size="0.9 0.8 0.3"/>
+            </geometry>
+        </collision>
+    </link>
+    <gazebo reference="base_link">
+        <material>Gazebo/Blue</material>
+    </gazebo>
+    <joint name="wheel_left_joint" type="fixed">
+        <parent link="base_link"/>
+        <child link="wheel_left_link"/>
+        <origin xyz="0 1 0" rpy="1.57 0 0"/>
+    </joint>
+    <link name="wheel_left_link">
+        <inertial>
+            <origin xyz="0 0 0"/>
+            <mass value="1.0"/>
+            <inertia ixx="1.0" ixy="0.0"   ixz="0.0"
+                               iyy="100.0" iyz="0.0"
+                                           izz="1.0"/>
+        </inertial>
+        <visual>
+            <origin xyz="0 0 0"/>
+            <geometry>
+                <cylinder radius="${wheel_radius}" length="${wheel_thickness}"/>
+            </geometry>
+        </visual>
+        <collision>
+            <origin xyz="0 0 0"/>
+            <geometry>
+                <cylinder radius="${wheel_radius}" length="${wheel_thickness}"/>
+            </geometry>
+        </collision>
+    </link>
+    <joint name="wheel_right_joint" type="fixed">
+        <parent link="base_link"/>
+        <child link="wheel_right_link"/>
+        <origin xyz="0 -1 0" rpy="1.57 0 0"/>
+    </joint>
+    <link name="wheel_right_link">
+        <inertial>
+            <origin xyz="0 0 0"/>
+            <mass value="1.0"/>
+            <inertia ixx="1.0" ixy="0.0"   ixz="0.0"
+                               iyy="100.0" iyz="0.0"
+                                           izz="1.0" />
+        </inertial>
+        <visual>
+            <origin xyz="0 0 0"/>
+            <geometry>
+                <cylinder radius="${wheel_radius}" length="${wheel_thickness}"/>
+            </geometry>
+        </visual>
+        <collision>
+            <origin xyz="0 0 0"/>
+            <geometry>
+                <cylinder radius="${wheel_radius}" length="${wheel_thickness}"/>
+            </geometry>
+        </collision>
+    </link>
+    <joint name="caster_joint" type="fixed">
+        <parent link="base_link"/>
+        <child link="caster_link"/>
+        <origin xyz="-1 0 0" rpy="1.57 0 0"/>
+    </joint>
+    <link name="caster_link">
+        <inertial>
+            <origin xyz="0 0 0"/>
+            <mass value="1.0"/>
+            <inertia ixx="1.0" ixy="0.0"   ixz="0.0"
+                               iyy="100.0" iyz="0.0"
+                                           izz="1.0" />
+        </inertial>
+        <visual>
+            <origin xyz="0 0 0"/>
+            <geometry>
+                <cylinder radius="${wheel_radius}" length="${wheel_thickness}"/>
+            </geometry>
+        </visual>
+        <collision>
+            <origin xyz="0 0 0"/>
+            <geometry>
+                <cylinder radius="${wheel_radius}" length="${wheel_thickness}"/>
+            </geometry>
+        </collision>
+    </link>
 </robot>

Commit message: they're round

File: navi_model/urdf/navi.urdf.xacro (robot description, xacro)
@@ -12,5 +12,8 @@
     <xacro:property name="robot_weight" value="90.0"/>
     <xacro:property name="wheel_radius" value="0.127"/>
-    <xacro:property name="wheel_thickness" value="0.05"/>
+    <xacro:property name="wheel_thickness" value="0.050"/>
+    <xacro:property name="wheel_separation" value="0.711"/>
+    <xacro:property name="caster_radius" value="0.095"/>
+    <xacro:property name="caster_thickness" value="0.064"/>
     <link name="base_link">
         <inertial>
@@ -105,5 +108,5 @@
             <origin xyz="0 0 0"/>
             <geometry>
-                <cylinder radius="${wheel_radius}" length="${wheel_thickness}"/>
+                <cylinder radius="${caster_radius}" length="${caster_thickness}"/>
             </geometry>
         </visual>
@@ -111,5 +114,5 @@
             <origin xyz="0 0 0"/>
             <geometry>
-                <cylinder radius="${wheel_radius}" length="${wheel_thickness}"/>
+                <cylinder radius="${caster_radius}" length="${caster_thickness}"/>
             </geometry>
         </collision>

Commit message: added wheel separation

File: navi_model/urdf/navi.urdf.xacro (robot description, xacro)
@@ -12,6 +12,6 @@
     <xacro:property name="robot_weight" value="90.0"/>
     <xacro:property name="wheel_radius" value="0.127"/>
-    <xacro:property name="wheel_thickness" value="0.050"/>
-    <xacro:property name="wheel_separation" value="0.711"/>
+    <xacro:property name="wheel_thickness" value="0.150"/>
+    <xacro:property name="wheel_separation" value="1.000"/>
     <xacro:property name="caster_radius" value="0.095"/>
     <xacro:property name="caster_thickness" value="0.064"/>
@@ -43,5 +43,5 @@
         <parent link="base_link"/>
         <child link="wheel_left_link"/>
-        <origin xyz="0 1 0" rpy="1.57 0 0"/>
+        <origin xyz="0 ${wheel_separation/2} 0" rpy="1.57 0 0"/>
     </joint>
     <link name="wheel_left_link">
@@ -69,5 +69,5 @@
         <parent link="base_link"/>
         <child link="wheel_right_link"/>
-        <origin xyz="0 -1 0" rpy="1.57 0 0"/>
+        <origin xyz="0 ${-wheel_separation/2} 0" rpy="1.57 0 0"/>
     </joint>
     <link name="wheel_right_link">

Commit message: fixed ground clearance

File: navi_model/urdf/navi.urdf.xacro (robot description, xacro)
@@ -14,4 +14,5 @@
     <xacro:property name="wheel_thickness" value="0.150"/>
     <xacro:property name="wheel_separation" value="1.000"/>
+    <xacro:property name="robot_clearance" value="0.170"/>
     <xacro:property name="caster_radius" value="0.095"/>
     <xacro:property name="caster_thickness" value="0.064"/>
@@ -43,5 +44,5 @@
         <parent link="base_link"/>
         <child link="wheel_left_link"/>
-        <origin xyz="0 ${wheel_separation/2} 0" rpy="1.57 0 0"/>
+        <origin xyz="0 ${wheel_separation/2} ${-robot_clearance}" rpy="${PI/2} 0 0"/>
     </joint>
     <link name="wheel_left_link">
@@ -69,5 +70,5 @@
         <parent link="base_link"/>
         <child link="wheel_right_link"/>
-        <origin xyz="0 ${-wheel_separation/2} 0" rpy="1.57 0 0"/>
+        <origin xyz="0 ${-wheel_separation/2} ${-robot_clearance}" rpy="${PI/2} 0 0"/>
     </joint>
     <link name="wheel_right_link">
@@ -95,5 +96,6 @@
         <parent link="base_link"/>
         <child link="caster_link"/>
-        <origin xyz="-1 0 0" rpy="1.57 0 0"/>
+        <origin xyz="-1 0 ${-robot_clearance-(wheel_radius-caster_radius)}"
+                rpy="${PI/2} 0 0"/>
     </joint>
     <link name="caster_link">

Commit message: front wheels right

File: navi_model/urdf/navi.urdf.xacro (robot description, xacro)
@@ -41,8 +41,9 @@
         <material>Gazebo/Blue</material>
     </gazebo>
-    <joint name="wheel_left_joint" type="fixed">
+    <joint name="wheel_left_joint" type="continuous">
         <parent link="base_link"/>
         <child link="wheel_left_link"/>
         <origin xyz="0 ${wheel_separation/2} ${-robot_clearance}" rpy="${PI/2} 0 0"/>
+        <axis xyz="0 0 1"/>
     </joint>
     <link name="wheel_left_link">
@@ -67,8 +68,9 @@
         </collision>
     </link>
-    <joint name="wheel_right_joint" type="fixed">
+    <joint name="wheel_right_joint" type="continuous">
         <parent link="base_link"/>
         <child link="wheel_right_link"/>
         <origin xyz="0 ${-wheel_separation/2} ${-robot_clearance}" rpy="${PI/2} 0 0"/>
+        <axis xyz="0 0 1"/>
     </joint>
     <link name="wheel_right_link">
@@ -120,3 +122,18 @@
         </collision>
     </link>
+    <gazebo>
+        <controller:diffdrive_plugin name="differential_drive_controller" plugin="libdiffdrive_plugin.so">
+            <alwaysOn>true</alwaysOn>
+            <update>100</update>
+            <updateRate>100.0</updateRate>
+            <torque>1000</torque>
+            <wheelSeparation>${wheel_separation}</wheelSeparation>
+            <wheelDiameter>${wheel_radius*2}</wheelDiameter>
+            <robotNamespace>/</robotNamespace>
+            <topicName>drive/cmd_vel</topicName>
+            <leftJoint>wheel_left_joint</leftJoint>
+            <rightJoint>wheel_right_joint</rightJoint>
+            <interface:position name="drive_iface"/>
+        </controller:diffdrive_plugin>
+    </gazebo>
 </robot>

Commit message: added intermediate caster_pivot_link

File: navi_model/urdf/navi.urdf.xacro (robot description, xacro)
@@ -95,9 +95,22 @@
         </collision>
     </link>
-    <joint name="caster_joint" type="fixed">
+    <joint name="caster_pivot_joint" type="fixed">
         <parent link="base_link"/>
-        <child link="caster_link"/>
+        <child link="caster_pivot_link"/>
         <origin xyz="-1 0 ${-robot_clearance-(wheel_radius-caster_radius)}"
                 rpy="${PI/2} 0 0"/>
+    </joint>
+    <link name="caster_pivot_link">
+        <inertial>
+            <mass value="${EPS}"/>
+            <inertia ixx="${EPS}" ixy="0"      ixz="0"
+                                  iyy="${EPS}" iyz="0"
+                                               izz="${EPS}"/>
+        </inertial>
+    </link>
+    <joint name="caster_joint" type="continuous">
+        <parent link="caster_pivot_link"/>
+        <child link="caster_link"/>
+        <axis xyz="0 0 1"/>
     </joint>
     <link name="caster_link">

Commit message: used 'correct' wheel/caster MOI

File: navi_model/urdf/navi.urdf.xacro (robot description, xacro)
@@ -14,7 +14,9 @@
     <xacro:property name="wheel_thickness" value="0.150"/>
     <xacro:property name="wheel_separation" value="1.000"/>
+    <xacro:property name="wheel_mass" value="3.175"/>
     <xacro:property name="robot_clearance" value="0.170"/>
     <xacro:property name="caster_radius" value="0.095"/>
     <xacro:property name="caster_thickness" value="0.064"/>
+    <xacro:property name="caster_mass" value="2.268"/>
     <link name="base_link">
         <inertial>
@@ -50,8 +52,8 @@
         <inertial>
             <origin xyz="0 0 0"/>
-            <mass value="1.0"/>
-            <inertia ixx="1.0" ixy="0.0"   ixz="0.0"
-                               iyy="100.0" iyz="0.0"
-                                           izz="1.0"/>
+            <mass value="${wheel_mass}"/>
+            <inertia ixx="${wheel_mass*(3*wheel_radius*wheel_radius + wheel_thickness*wheel_thickness)}" ixy="0.0" ixz="0.0"
+                     iyy="${wheel_mass*(3*wheel_radius*wheel_radius + wheel_thickness*wheel_thickness)}" iyz="0.0"
+                     izz="${wheel_mass*wheel_radius*wheel_radius/2}"/>
         </inertial>
         <visual>
@@ -77,8 +79,8 @@
         <inertial>
             <origin xyz="0 0 0"/>
-            <mass value="1.0"/>
-            <inertia ixx="1.0" ixy="0.0"   ixz="0.0"
-                               iyy="100.0" iyz="0.0"
-                                           izz="1.0" />
+            <mass value="${wheel_mass}"/>
+            <inertia ixx="${wheel_mass*(3*wheel_radius*wheel_radius + wheel_thickness*wheel_thickness)}" ixy="0.0" ixz="0.0"
+                     iyy="${wheel_mass*(3*wheel_radius*wheel_radius + wheel_thickness*wheel_thickness)}" iyz="0.0"
+                     izz="${wheel_mass*wheel_radius*wheel_radius/2}"/>
         </inertial>
         <visual>
@@ -95,9 +97,12 @@
         </collision>
     </link>
-    <joint name="caster_pivot_joint" type="fixed">
+    <joint name="caster_pivot_joint" type="continuous">
         <parent link="base_link"/>
         <child link="caster_pivot_link"/>
         <origin xyz="-1 0 ${-robot_clearance-(wheel_radius-caster_radius)}"
                 rpy="${PI/2} 0 0"/>
+        <axis xyz="0 1 0"/>
+        <limit effort="100" velocity="100" k_velocity="0" />
+        <joint_properties damping="0.0" friction="0.0" />
     </joint>
     <link name="caster_pivot_link">
@@ -112,4 +117,5 @@
         <parent link="caster_pivot_link"/>
         <child link="caster_link"/>
+        <origin xyz="0 0 0"/>
         <axis xyz="0 0 1"/>
     </joint>
@@ -117,8 +123,8 @@
         <inertial>
             <origin xyz="0 0 0"/>
-            <mass value="1.0"/>
-            <inertia ixx="1.0" ixy="0.0"   ixz="0.0"
-                               iyy="100.0" iyz="0.0"
-                                           izz="1.0" />
+            <mass value="${caster_mass}"/>
+            <inertia ixx="${caster_mass*(3*caster_radius*caster_radius + caster_thickness*caster_thickness)}" ixy="0.0" ixz="0.0"
+                     iyy="${caster_mass*(3*caster_radius*caster_radius + caster_thickness*caster_thickness)}" iyz="0.0"
+                     izz="${caster_mass*caster_radius*caster_radius/2}"/>
         </inertial>
         <visual>

Commit message: removed extra zero origins

File: navi_model/urdf/navi.urdf.xacro (robot description, xacro)
@@ -21,5 +21,4 @@
     <link name="base_link">
         <inertial>
-            <origin xyz="0 0 0"/>
             <mass value="1.0"/>
             <inertia ixx="1.0" ixy="0.0"   ixz="0.0"
@@ -28,5 +27,4 @@
         </inertial>
         <visual>
-            <origin xyz="0 0 0"/>
             <geometry>
                 <box size="0.9 0.8 0.3"/>
@@ -34,5 +32,4 @@
         </visual>
         <collision>
-            <origin xyz="0 0 0"/>
             <geometry>
                 <box size="0.9 0.8 0.3"/>
@@ -51,5 +48,4 @@
     <link name="wheel_left_link">
         <inertial>
-            <origin xyz="0 0 0"/>
             <mass value="${wheel_mass}"/>
             <inertia ixx="${wheel_mass*(3*wheel_radius*wheel_radius + wheel_thickness*wheel_thickness)}" ixy="0.0" ixz="0.0"
@@ -58,5 +54,4 @@
         </inertial>
         <visual>
-            <origin xyz="0 0 0"/>
             <geometry>
                 <cylinder radius="${wheel_radius}" length="${wheel_thickness}"/>
@@ -64,5 +59,4 @@
         </visual>
         <collision>
-            <origin xyz="0 0 0"/>
             <geometry>
                 <cylinder radius="${wheel_radius}" length="${wheel_thickness}"/>
@@ -78,5 +72,4 @@
     <link name="wheel_right_link">
         <inertial>
-            <origin xyz="0 0 0"/>
             <mass value="${wheel_mass}"/>
             <inertia ixx="${wheel_mass*(3*wheel_radius*wheel_radius + wheel_thickness*wheel_thickness)}" ixy="0.0" ixz="0.0"
@@ -85,5 +78,4 @@
         </inertial>
         <visual>
-            <origin xyz="0 0 0"/>
             <geometry>
                 <cylinder radius="${wheel_radius}" length="${wheel_thickness}"/>
@@ -91,5 +83,4 @@
         </visual>
         <collision>
-            <origin xyz="0 0 0"/>
             <geometry>
                 <cylinder radius="${wheel_radius}" length="${wheel_thickness}"/>
@@ -122,5 +113,4 @@
     <link name="caster_link">
         <inertial>
-            <origin xyz="0 0 0"/>
             <mass value="${caster_mass}"/>
             <inertia ixx="${caster_mass*(3*caster_radius*caster_radius + caster_thickness*caster_thickness)}" ixy="0.0" ixz="0.0"
@@ -129,5 +119,7 @@
         </inertial>
         <visual>
-            <origin xyz="0 0 0"/>
+            <inertia ixx="${wheel_mass*(3*wheel_radius*wheel_radius + wheel_thickness*wheel_thickness)}" ixy="0.0" ixz="0.0"
+                     iyy="${wheel_mass*(3*wheel_radius*wheel_radius + wheel_thickness*wheel_thickness)}" iyz="0.0"
+                     izz="${wheel_mass*wheel_radius*wheel_radius/2}"/>
             <geometry>
                 <cylinder radius="${caster_radius}" length="${caster_thickness}"/>
@@ -135,5 +127,4 @@
         </visual>
         <collision>
-            <origin xyz="0 0 0"/>
             <geometry>
                 <cylinder radius="${caster_radius}" length="${caster_thickness}"/>

Commit message: almost there (with the caster, even)

File: navi_model/urdf/navi.urdf.xacro (robot description, xacro)
@@ -12,11 +12,15 @@
     <xacro:property name="robot_weight" value="90.0"/>
     <xacro:property name="wheel_radius" value="0.127"/>
-    <xacro:property name="wheel_thickness" value="0.150"/>
-    <xacro:property name="wheel_separation" value="1.000"/>
+    <xacro:property name="wheel_thickness" value="0.0762"/>
+    <xacro:property name="wheel_separation" value="0.70386"/>
     <xacro:property name="wheel_mass" value="3.175"/>
-    <xacro:property name="robot_clearance" value="0.170"/>
-    <xacro:property name="caster_radius" value="0.095"/>
-    <xacro:property name="caster_thickness" value="0.064"/>
+    <xacro:property name="robot_clearance" value="0.3937"/>
+    <xacro:property name="caster_radius" value="0.1143"/>
+    <xacro:property name="caster_thickness" value="0.0508"/>
+    <xacro:property name="caster_separation" value="0.53388"/>
+    <xacro:property name="caster_clearance" value="0.254"/>
     <xacro:property name="caster_mass" value="2.268"/>
+    <xacro:property name="caster_offset_height" value="0.1524"/>
+    <xacro:property name="caster_offset_axis" value="0.0889"/>
     <link name="base_link">
         <inertial>
@@ -91,9 +95,7 @@
         <parent link="base_link"/>
         <child link="caster_pivot_link"/>
-        <origin xyz="-1 0 ${-robot_clearance-(wheel_radius-caster_radius)}"
+        <origin xyz="${-caster_separation} 0 ${-caster_clearance)}"
                 rpy="${PI/2} 0 0"/>
         <axis xyz="0 1 0"/>
-        <limit effort="100" velocity="100" k_velocity="0" />
-        <joint_properties damping="0.0" friction="0.0" />
     </joint>
     <link name="caster_pivot_link">
@@ -105,8 +107,9 @@
         </inertial>
     </link>
-    <joint name="caster_joint" type="continuous">
+    <!-- TODO: Why can't I make this continuous? -->
+    <joint name="caster_joint" type="fixed">
         <parent link="caster_pivot_link"/>
         <child link="caster_link"/>
-        <origin xyz="0 0 0"/>
+        <origin xyz="${-caster_offset_axis} ${-caster_offset_height} 0"/>
         <axis xyz="0 0 1"/>
     </joint>

Commit message: added the low poly model

File: navi_model/urdf/navi.urdf.xacro (robot description, xacro)
@@ -15,4 +15,5 @@
     <xacro:property name="wheel_separation" value="0.70386"/>
     <xacro:property name="wheel_mass" value="3.175"/>
+    <xacro:property name="wheel_torque" value="10"/>
     <xacro:property name="robot_clearance" value="0.3937"/>
     <xacro:property name="caster_radius" value="0.1143"/>
@@ -23,4 +24,5 @@
     <xacro:property name="caster_offset_height" value="0.1524"/>
     <xacro:property name="caster_offset_axis" value="0.0889"/>
+    <xacro:property name="mesh_offset" value="-0.60 0.300 -0.50"/>
     <link name="base_link">
         <inertial>
@@ -31,6 +33,7 @@
         </inertial>
         <visual>
+            <origin xyz="${mesh_offset}" rpy="${PI/2} 0 0"/>
             <geometry>
-                <box size="0.9 0.8 0.3"/>
+                <mesh filename="package://navi_model/meshes/frame.stl" scale="0.001 0.001 0.001"/>
             </geometry>
         </visual>
@@ -101,5 +104,5 @@
     <link name="caster_pivot_link">
         <inertial>
-            <mass value="${EPS}"/>
+            <mass value="${caster_mass}"/>
             <inertia ixx="${EPS}" ixy="0"      ixz="0"
                                   iyy="${EPS}" iyz="0"
@@ -140,5 +143,5 @@
             <update>100</update>
             <updateRate>100.0</updateRate>
-            <torque>1000</torque>
+            <torque>${wheel_torque}</torque>
             <wheelSeparation>${wheel_separation}</wheelSeparation>
             <wheelDiameter>${wheel_radius*2}</wheelDiameter>
