Commit message: moved wheels into xacro macros

File: navi_model/urdf/navi.urdf.xacro (robot description, xacro)
@@ -25,74 +25,57 @@
     <xacro:property name="caster_offset_axis" value="0.0889"/>
     <xacro:property name="mesh_offset" value="-0.60 0.300 -0.50"/>
-    <link name="base_link">
-        <inertial>
-            <mass value="1.0"/>
-            <inertia ixx="1.0" ixy="0.0"   ixz="0.0"
-                               iyy="100.0" iyz="0.0"
-                                           izz="1.0" />
-        </inertial>
-        <visual>
-            <origin xyz="${mesh_offset}" rpy="${PI/2} 0 0"/>
-            <geometry>
-                <mesh filename="package://navi_model/meshes/frame.stl" scale="0.001 0.001 0.001"/>
-            </geometry>
-        </visual>
-        <collision>
-            <geometry>
-                <box size="0.9 0.8 0.3"/>
-            </geometry>
-        </collision>
-    </link>
-    <gazebo reference="base_link">
-        <material>Gazebo/Blue</material>
-    </gazebo>
-    <joint name="wheel_left_joint" type="continuous">
-        <parent link="base_link"/>
-        <child link="wheel_left_link"/>
-        <origin xyz="0 ${wheel_separation/2} ${-robot_clearance}" rpy="${PI/2} 0 0"/>
-        <axis xyz="0 0 1"/>
-    </joint>
-    <link name="wheel_left_link">
-        <inertial>
-            <mass value="${wheel_mass}"/>
-            <inertia ixx="${wheel_mass*(3*wheel_radius*wheel_radius + wheel_thickness*wheel_thickness)}" ixy="0.0" ixz="0.0"
-                     iyy="${wheel_mass*(3*wheel_radius*wheel_radius + wheel_thickness*wheel_thickness)}" iyz="0.0"
-                     izz="${wheel_mass*wheel_radius*wheel_radius/2}"/>
-        </inertial>
-        <visual>
-            <geometry>
-                <cylinder radius="${wheel_radius}" length="${wheel_thickness}"/>
-            </geometry>
-        </visual>
-        <collision>
-            <geometry>
-                <cylinder radius="${wheel_radius}" length="${wheel_thickness}"/>
-            </geometry>
-        </collision>
-    </link>
-    <joint name="wheel_right_joint" type="continuous">
-        <parent link="base_link"/>
-        <child link="wheel_right_link"/>
-        <origin xyz="0 ${-wheel_separation/2} ${-robot_clearance}" rpy="${PI/2} 0 0"/>
-        <axis xyz="0 0 1"/>
-    </joint>
-    <link name="wheel_right_link">
-        <inertial>
-            <mass value="${wheel_mass}"/>
-            <inertia ixx="${wheel_mass*(3*wheel_radius*wheel_radius + wheel_thickness*wheel_thickness)}" ixy="0.0" ixz="0.0"
-                     iyy="${wheel_mass*(3*wheel_radius*wheel_radius + wheel_thickness*wheel_thickness)}" iyz="0.0"
-                     izz="${wheel_mass*wheel_radius*wheel_radius/2}"/>
-        </inertial>
-        <visual>
-            <geometry>
-                <cylinder radius="${wheel_radius}" length="${wheel_thickness}"/>
-            </geometry>
-        </visual>
-        <collision>
-            <geometry>
-                <cylinder radius="${wheel_radius}" length="${wheel_thickness}"/>
-            </geometry>
-        </collision>
-    </link>
+    <xacro:macro name="chassis">
+        <link name="base_link">
+            <inertial>
+                <mass value="1.0"/>
+                <inertia ixx="1.0" ixy="0.0"   ixz="0.0"
+                                   iyy="100.0" iyz="0.0"
+                                               izz="1.0" />
+            </inertial>
+            <visual>
+                <origin xyz="${mesh_offset}" rpy="${PI/2} 0 0"/>
+                <geometry>
+                    <mesh filename="package://navi_model/meshes/frame.stl" scale="0.001 0.001 0.001"/>
+                </geometry>
+            </visual>
+            <collision>
+                <geometry>
+                    <box size="0.9 0.8 0.3"/>
+                </geometry>
+            </collision>
+        </link>
+        <gazebo reference="base_link">
+            <material>Gazebo/Blue</material>
+        </gazebo>
+    </xacro:macro>
+    <xacro:macro name="wheel" params="side sign">
+        <joint name="wheel_${side}_joint" type="continuous">
+            <parent link="base_link"/>
+            <child link="wheel_${side}_link"/>
+            <origin xyz="0 ${sign*wheel_separation/2} ${-robot_clearance}" rpy="${PI/2} 0 0"/>
+            <axis xyz="0 0 1"/>
+        </joint>
+        <link name="wheel_${side}_link">
+            <inertial>
+                <mass value="${wheel_mass}"/>
+                <inertia ixx="${wheel_mass*(3*wheel_radius*wheel_radius + wheel_thickness*wheel_thickness)}" ixy="0.0" ixz="0.0"
+                         iyy="${wheel_mass*(3*wheel_radius*wheel_radius + wheel_thickness*wheel_thickness)}" iyz="0.0"
+                         izz="${wheel_mass*wheel_radius*wheel_radius/2}"/>
+            </inertial>
+            <visual>
+                <geometry>
+                    <cylinder radius="${wheel_radius}" length="${wheel_thickness}"/>
+                </geometry>
+            </visual>
+            <collision>
+                <geometry>
+                    <cylinder radius="${wheel_radius}" length="${wheel_thickness}"/>
+                </geometry>
+            </collision>
+        </link>
+        <gazebo reference="wheel_${side}_link">
+            <material>Gazebo/Red</material>
+        </gazebo>
+    </xacro:macro>
     <joint name="caster_pivot_joint" type="continuous">
         <parent link="base_link"/>
@@ -138,4 +121,10 @@
         </collision>
     </link>
+    <gazebo reference="caster_link">
+        <material>Gazebo/Red</material>
+    </gazebo>
+    <xacro:chassis/>
+    <xacro:wheel sign="-1" side="left"/>
+    <xacro:wheel sign="+1" side="right"/>
     <gazebo>
         <controller:diffdrive_plugin name="differential_drive_controller" plugin="libdiffdrive_plugin.so">

Commit message: moved the caster into an xacro macro

File: navi_model/urdf/navi.urdf.xacro (robot description, xacro)
@@ -78,53 +78,56 @@
         </gazebo>
     </xacro:macro>
-    <joint name="caster_pivot_joint" type="continuous">
-        <parent link="base_link"/>
-        <child link="caster_pivot_link"/>
-        <origin xyz="${-caster_separation} 0 ${-caster_clearance)}"
-                rpy="${PI/2} 0 0"/>
-        <axis xyz="0 1 0"/>
-    </joint>
-    <link name="caster_pivot_link">
-        <inertial>
-            <mass value="${caster_mass}"/>
-            <inertia ixx="${EPS}" ixy="0"      ixz="0"
-                                  iyy="${EPS}" iyz="0"
-                                               izz="${EPS}"/>
-        </inertial>
-    </link>
-    <!-- TODO: Why can't I make this continuous? -->
-    <joint name="caster_joint" type="fixed">
-        <parent link="caster_pivot_link"/>
-        <child link="caster_link"/>
-        <origin xyz="${-caster_offset_axis} ${-caster_offset_height} 0"/>
-        <axis xyz="0 0 1"/>
-    </joint>
-    <link name="caster_link">
-        <inertial>
-            <mass value="${caster_mass}"/>
-            <inertia ixx="${caster_mass*(3*caster_radius*caster_radius + caster_thickness*caster_thickness)}" ixy="0.0" ixz="0.0"
-                     iyy="${caster_mass*(3*caster_radius*caster_radius + caster_thickness*caster_thickness)}" iyz="0.0"
-                     izz="${caster_mass*caster_radius*caster_radius/2}"/>
-        </inertial>
-        <visual>
-            <inertia ixx="${wheel_mass*(3*wheel_radius*wheel_radius + wheel_thickness*wheel_thickness)}" ixy="0.0" ixz="0.0"
-                     iyy="${wheel_mass*(3*wheel_radius*wheel_radius + wheel_thickness*wheel_thickness)}" iyz="0.0"
-                     izz="${wheel_mass*wheel_radius*wheel_radius/2}"/>
-            <geometry>
-                <cylinder radius="${caster_radius}" length="${caster_thickness}"/>
-            </geometry>
-        </visual>
-        <collision>
-            <geometry>
-                <cylinder radius="${caster_radius}" length="${caster_thickness}"/>
-            </geometry>
-        </collision>
-    </link>
-    <gazebo reference="caster_link">
-        <material>Gazebo/Red</material>
-    </gazebo>
+    <xacro:macro name="caster">
+        <joint name="caster_pivot_joint" type="continuous">
+            <parent link="base_link"/>
+            <child link="caster_pivot_link"/>
+            <origin xyz="${-caster_separation} 0 ${-caster_clearance)}"
+                    rpy="${PI/2} 0 0"/>
+            <axis xyz="0 1 0"/>
+        </joint>
+        <link name="caster_pivot_link">
+            <inertial>
+                <mass value="${caster_mass}"/>
+                <inertia ixx="${EPS}" ixy="0"      ixz="0"
+                                      iyy="${EPS}" iyz="0"
+                                                   izz="${EPS}"/>
+            </inertial>
+        </link>
+        <!-- TODO: Why can't I make this continuous? -->
+        <joint name="caster_joint" type="fixed">
+            <parent link="caster_pivot_link"/>
+            <child link="caster_link"/>
+            <origin xyz="${-caster_offset_axis} ${-caster_offset_height} 0"/>
+            <axis xyz="0 0 1"/>
+        </joint>
+        <link name="caster_link">
+            <inertial>
+                <mass value="${caster_mass}"/>
+                <inertia ixx="${caster_mass*(3*caster_radius*caster_radius + caster_thickness*caster_thickness)}" ixy="0.0" ixz="0.0"
+                         iyy="${caster_mass*(3*caster_radius*caster_radius + caster_thickness*caster_thickness)}" iyz="0.0"
+                         izz="${caster_mass*caster_radius*caster_radius/2}"/>
+            </inertial>
+            <visual>
+                <inertia ixx="${wheel_mass*(3*wheel_radius*wheel_radius + wheel_thickness*wheel_thickness)}" ixy="0.0" ixz="0.0"
+                         iyy="${wheel_mass*(3*wheel_radius*wheel_radius + wheel_thickness*wheel_thickness)}" iyz="0.0"
+                         izz="${wheel_mass*wheel_radius*wheel_radius/2}"/>
+                <geometry>
+                    <cylinder radius="${caster_radius}" length="${caster_thickness}"/>
+                </geometry>
+            </visual>
+            <collision>
+                <geometry>
+                    <cylinder radius="${caster_radius}" length="${caster_thickness}"/>
+                </geometry>
+            </collision>
+        </link>
+        <gazebo reference="caster_link">
+            <material>Gazebo/Red</material>
+        </gazebo>
+    </xacro:macro>
     <xacro:chassis/>
     <xacro:wheel sign="-1" side="left"/>
     <xacro:wheel sign="+1" side="right"/>
+    <xacro:caster/>
     <gazebo>
         <controller:diffdrive_plugin name="differential_drive_controller" plugin="libdiffdrive_plugin.so">

Commit message: added ground truth localization info

File: navi_model/urdf/navi.urdf.xacro (robot description, xacro)
@@ -126,22 +126,39 @@
         </gazebo>
     </xacro:macro>
+    <xacro:macro name="gazebo_drive">
+        <gazebo>
+            <controller:diffdrive_plugin name="differential_drive_controller" plugin="libdiffdrive_plugin.so">
+                <alwaysOn>true</alwaysOn>
+                <update>100</update>
+                <updateRate>100.0</updateRate>
+                <torque>${wheel_torque}</torque>
+                <wheelSeparation>${wheel_separation}</wheelSeparation>
+                <wheelDiameter>${wheel_radius*2}</wheelDiameter>
+                <robotNamespace>/</robotNamespace>
+                <topicName>drive/cmd_vel</topicName>
+                <leftJoint>wheel_left_joint</leftJoint>
+                <rightJoint>wheel_right_joint</rightJoint>
+                <interface:position name="drive_iface"/>
+            </controller:diffdrive_plugin>
+        </gazebo>
+    </xacro:macro>
+    <xacro:macro name="gazebo_localization">
+        <gazebo>
+            <controller:gazebo_ros_p3d name="gps_controller" plugin="libgazebo_ros_p3d.so">
+                <alwaysOn>true</alwaysOn>
+                <updateRate>60</updateRate>
+                <bodyName>base_link</bodyName>
+                <topicName>ground_truth</topicName>
+                <gaussianNoise>0.0</gaussianNoise>
+                <frameName>/map</frameName>
+                <interface:position name="gps_iface"/>
+            </controller:gazebo_ros_p3d>
+            <canonicalBody>base_link</canonicalBody>
+        </gazebo>
+    </xacro:macro>
     <xacro:chassis/>
     <xacro:wheel sign="-1" side="left"/>
     <xacro:wheel sign="+1" side="right"/>
     <xacro:caster/>
-    <gazebo>
-        <controller:diffdrive_plugin name="differential_drive_controller" plugin="libdiffdrive_plugin.so">
-            <alwaysOn>true</alwaysOn>
-            <update>100</update>
-            <updateRate>100.0</updateRate>
-            <torque>${wheel_torque}</torque>
-            <wheelSeparation>${wheel_separation}</wheelSeparation>
-            <wheelDiameter>${wheel_radius*2}</wheelDiameter>
-            <robotNamespace>/</robotNamespace>
-            <topicName>drive/cmd_vel</topicName>
-            <leftJoint>wheel_left_joint</leftJoint>
-            <rightJoint>wheel_right_joint</rightJoint>
-            <interface:position name="drive_iface"/>
-        </controller:diffdrive_plugin>
-    </gazebo>
+    <xacro:gazebo_drive/>
 </robot>

Commit message: hack to work around diffdrive_plugin's poor design

File: navi_model/urdf/navi.urdf.xacro (robot description, xacro)
@@ -25,5 +25,22 @@
     <xacro:property name="caster_offset_axis" value="0.0889"/>
     <xacro:property name="mesh_offset" value="-0.60 0.300 -0.50"/>
+    <xacro:macro name="weightless">
+        <inertial>
+            <mass value="${EPS}"/>
+            <inertia ixx="${EPS}" ixy="0"      ixz="0"
+                                  iyy="${EPS}" iyz="0"
+                                               izz="${EPS}"/>
+        </inertial>
+    </xacro:macro>
     <xacro:macro name="chassis">
+        <link name="base_footprint">
+            <origin xyz="0 0 ${-robot_clearance - wheel_radius}"/>
+            <xacro:weightless/>
+        </link>
+        <joint name="base_link_joint" type="fixed">
+            <parent link="base_footprint"/>
+            <child link="base_link"/>
+            <origin xyz="0 0 ${robot_clearance + wheel_radius}"/>
+        </joint>
         <link name="base_link">
             <inertial>

Commit message: temporarily fixed the simulation issues

File: navi_model/urdf/navi.urdf.xacro (robot description, xacro)
@@ -34,13 +34,4 @@
     </xacro:macro>
     <xacro:macro name="chassis">
-        <link name="base_footprint">
-            <origin xyz="0 0 ${-robot_clearance - wheel_radius}"/>
-            <xacro:weightless/>
-        </link>
-        <joint name="base_link_joint" type="fixed">
-            <parent link="base_footprint"/>
-            <child link="base_link"/>
-            <origin xyz="0 0 ${robot_clearance + wheel_radius}"/>
-        </joint>
         <link name="base_link">
             <inertial>
@@ -65,4 +56,12 @@
             <material>Gazebo/Blue</material>
         </gazebo>
+        <joint name="base_link_joint" type="fixed">
+            <parent link="base_link"/>
+            <child link="base_footprint"/>
+            <origin xyz="0 0 ${-robot_clearance - wheel_radius}"/>
+        </joint>
+        <link name="base_footprint">
+            <xacro:weightless/>
+        </link>
     </xacro:macro>
     <xacro:macro name="wheel" params="side sign">
