Commit message: working from the pr2 model

File: navi_model/urdf/navi.urdf.xacro (robot description, xacro)
@@ -1,181 +1,52 @@
 <?xml version="1.0"?>
-<robot xmlns:body="http://playerstage.sourceforge.net/gazebo/xmlschema/#body"
-       xmlns:controller="http://playerstage.sourceforge.net/gazebo/xmlschema/#controller"
-       xmlns:geom="http://playerstage.sourceforge.net/gazebo/xmlschema/#geom"
+<robot xmlns:controller="http://playerstage.sourceforge.net/gazebo/xmlschema/#controller"
        xmlns:interface="http://playerstage.sourceforge.net/gazebo/xmlschema/#interface"
-       xmlns:joint="http://playerstage.sourceforge.net/gazebo/xmlschema/#slider"
-       xmlns:sensor="http://playerstage.sourceforge.net/gazebo/xmlschema/#sensor"
        xmlns:xacro="http://ros.org/wiki/xacro"
        name="navi">
-    <xacro:property name="EPS" value="0.000001"/>
-    <xacro:property name="PI" value="3.1415926535897931"/>
-    <xacro:property name="robot_weight" value="90.0"/>
-    <xacro:property name="wheel_radius" value="0.127"/>
-    <xacro:property name="wheel_thickness" value="0.0762"/>
-    <xacro:property name="wheel_separation" value="0.70386"/>
-    <xacro:property name="wheel_mass" value="3.175"/>
-    <xacro:property name="wheel_torque" value="10"/>
-    <xacro:property name="robot_clearance" value="0.3937"/>
-    <xacro:property name="caster_radius" value="0.1143"/>
-    <xacro:property name="caster_thickness" value="0.0508"/>
-    <xacro:property name="caster_separation" value="0.53388"/>
-    <xacro:property name="caster_clearance" value="0.254"/>
-    <xacro:property name="caster_mass" value="2.268"/>
-    <xacro:property name="caster_offset_height" value="0.1524"/>
-    <xacro:property name="caster_offset_axis" value="0.0889"/>
-    <xacro:property name="mesh_offset" value="-0.60 0.300 -0.50"/>
-    <xacro:macro name="weightless">
-        <inertial>
-            <mass value="${EPS}"/>
-            <inertia ixx="${EPS}" ixy="0"      ixz="0"
-                                  iyy="${EPS}" iyz="0"
-                                               izz="${EPS}"/>
-        </inertial>
-    </xacro:macro>
-    <xacro:macro name="chassis">
-        <link name="base_link">
-            <inertial>
-                <mass value="1.0"/>
-                <inertia ixx="1.0" ixy="0.0"   ixz="0.0"
-                                   iyy="100.0" iyz="0.0"
-                                               izz="1.0" />
-            </inertial>
-            <visual>
-                <origin xyz="${mesh_offset}" rpy="${PI/2} 0 0"/>
-                <geometry>
-                    <mesh filename="package://navi_model/meshes/frame.stl" scale="0.001 0.001 0.001"/>
-                </geometry>
-            </visual>
-            <collision>
-                <geometry>
-                    <box size="0.9 0.8 0.3"/>
-                </geometry>
-            </collision>
-        </link>
-        <gazebo reference="base_link">
-            <material>Gazebo/Blue</material>
-        </gazebo>
-        <joint name="base_link_joint" type="fixed">
-            <parent link="base_link"/>
-            <child link="base_footprint"/>
-            <origin xyz="0 0 ${-robot_clearance - wheel_radius}"/>
-        </joint>
-        <link name="base_footprint">
-            <xacro:weightless/>
-        </link>
-    </xacro:macro>
-    <xacro:macro name="wheel" params="side sign">
-        <joint name="wheel_${side}_joint" type="continuous">
-            <parent link="base_link"/>
-            <child link="wheel_${side}_link"/>
-            <origin xyz="0 ${sign*wheel_separation/2} ${-robot_clearance}" rpy="${PI/2} 0 0"/>
-            <axis xyz="0 0 1"/>
-        </joint>
-        <link name="wheel_${side}_link">
-            <inertial>
-                <mass value="${wheel_mass}"/>
-                <inertia ixx="${wheel_mass*(3*wheel_radius*wheel_radius + wheel_thickness*wheel_thickness)}" ixy="0.0" ixz="0.0"
-                         iyy="${wheel_mass*(3*wheel_radius*wheel_radius + wheel_thickness*wheel_thickness)}" iyz="0.0"
-                         izz="${wheel_mass*wheel_radius*wheel_radius/2}"/>
-            </inertial>
-            <visual>
-                <geometry>
-                    <cylinder radius="${wheel_radius}" length="${wheel_thickness}"/>
-                </geometry>
-            </visual>
-            <collision>
-                <geometry>
-                    <cylinder radius="${wheel_radius}" length="${wheel_thickness}"/>
-                </geometry>
-            </collision>
-        </link>
-        <gazebo reference="wheel_${side}_link">
-            <material>Gazebo/Red</material>
-        </gazebo>
-    </xacro:macro>
-    <xacro:macro name="caster">
-        <joint name="caster_pivot_joint" type="continuous">
-            <parent link="base_link"/>
-            <child link="caster_pivot_link"/>
-            <origin xyz="${-caster_separation} 0 ${-caster_clearance)}"
-                    rpy="${PI/2} 0 0"/>
-            <axis xyz="0 1 0"/>
-        </joint>
-        <link name="caster_pivot_link">
-            <inertial>
-                <mass value="${caster_mass}"/>
-                <inertia ixx="${EPS}" ixy="0"      ixz="0"
-                                      iyy="${EPS}" iyz="0"
-                                                   izz="${EPS}"/>
-            </inertial>
-        </link>
-        <!-- TODO: Why can't I make this continuous? -->
-        <joint name="caster_joint" type="fixed">
-            <parent link="caster_pivot_link"/>
-            <child link="caster_link"/>
-            <origin xyz="${-caster_offset_axis} ${-caster_offset_height} 0"/>
-            <axis xyz="0 0 1"/>
-        </joint>
-        <link name="caster_link">
-            <inertial>
-                <mass value="${caster_mass}"/>
-                <inertia ixx="${caster_mass*(3*caster_radius*caster_radius + caster_thickness*caster_thickness)}" ixy="0.0" ixz="0.0"
-                         iyy="${caster_mass*(3*caster_radius*caster_radius + caster_thickness*caster_thickness)}" iyz="0.0"
-                         izz="${caster_mass*caster_radius*caster_radius/2}"/>
-            </inertial>
-            <visual>
-                <inertia ixx="${wheel_mass*(3*wheel_radius*wheel_radius + wheel_thickness*wheel_thickness)}" ixy="0.0" ixz="0.0"
-                         iyy="${wheel_mass*(3*wheel_radius*wheel_radius + wheel_thickness*wheel_thickness)}" iyz="0.0"
-                         izz="${wheel_mass*wheel_radius*wheel_radius/2}"/>
-                <geometry>
-                    <cylinder radius="${caster_radius}" length="${caster_thickness}"/>
-                </geometry>
-            </visual>
-            <collision>
-                <geometry>
-                    <cylinder radius="${caster_radius}" length="${caster_thickness}"/>
-                </geometry>
-            </collision>
-        </link>
-        <gazebo reference="caster_link">
-            <material>Gazebo/Red</material>
-        </gazebo>
-    </xacro:macro>
-    <xacro:macro name="gazebo_drive">
-        <gazebo>
-            <controller:diffdrive_plugin name="differential_drive_controller" plugin="libdiffdrive_plugin.so">
-                <alwaysOn>true</alwaysOn>
-                <update>100</update>
-                <updateRate>100.0</updateRate>
-                <torque>${wheel_torque}</torque>
-                <wheelSeparation>${wheel_separation}</wheelSeparation>
-                <wheelDiameter>${wheel_radius*2}</wheelDiameter>
-                <robotNamespace>/</robotNamespace>
-                <topicName>drive/cmd_vel</topicName>
-                <leftJoint>wheel_left_joint</leftJoint>
-                <rightJoint>wheel_right_joint</rightJoint>
-                <interface:position name="drive_iface"/>
-            </controller:diffdrive_plugin>
-        </gazebo>
-    </xacro:macro>
-    <xacro:macro name="gazebo_localization">
-        <gazebo>
-            <controller:gazebo_ros_p3d name="gps_controller" plugin="libgazebo_ros_p3d.so">
-                <alwaysOn>true</alwaysOn>
-                <updateRate>60</updateRate>
-                <bodyName>base_link</bodyName>
-                <topicName>ground_truth</topicName>
-                <gaussianNoise>0.0</gaussianNoise>
-                <frameName>/map</frameName>
-                <interface:position name="gps_iface"/>
-            </controller:gazebo_ros_p3d>
-            <canonicalBody>base_link</canonicalBody>
-        </gazebo>
-    </xacro:macro>
-    <xacro:chassis/>
-    <xacro:wheel sign="-1" side="left"/>
-    <xacro:wheel sign="+1" side="right"/>
-    <xacro:caster/>
-    <xacro:gazebo_drive/>
-    <xacro:gazebo_localization/>
+    <!-- The following included files set up definitions of parts of the robot body -->
+    <!-- misc common stuff? -->
+    <include filename="$(find pr2_description)/urdf/common.xacro" />
+    <!-- PR2 Arm -->
+    <include filename="$(find pr2_description)/urdf/shoulder_v0/shoulder.urdf.xacro" />
+    <include filename="$(find pr2_description)/urdf/upper_arm_v0/upper_arm.urdf.xacro" />
+    <include filename="$(find pr2_description)/urdf/forearm_v0/forearm.urdf.xacro" />
+    <!-- PR2 gripper -->
+    <include filename="$(find pr2_description)/urdf/gripper_v0/gripper.urdf.xacro" />
+    <!-- PR2 head -->
+    <include filename="$(find pr2_description)/urdf/head_v0/head.urdf.xacro" />
+    <!-- PR2 tilting laser mount -->
+    <include filename="$(find pr2_description)/urdf/tilting_laser_v0/tilting_laser.urdf.xacro" />
+    <!-- PR2 torso -->
+    <include filename="$(find pr2_description)/urdf/torso_v0/torso.urdf.xacro" />
+    <!-- PR2 base -->
+    <include filename="$(find pr2_description)/urdf/base_v0/base.urdf.xacro" />
+    <!-- Head sensors -->
+    <include filename="$(find pr2_description)/urdf/sensors/head_sensor_package.urdf.xacro" />
+    <include filename="$(find pr2_description)/urdf/sensors/kinect_prosilica_camera.urdf.xacro" />
+    <!-- Camera sensors -->
+    <include filename="$(find pr2_description)/urdf/sensors/wge100_camera.urdf.xacro" />
+    <!-- Texture projector -->
+    <include filename="$(find pr2_description)/urdf/sensors/projector_wg6802418.urdf.xacro" />
+    <!-- generic simulator_gazebo plugins for starting mechanism control, ros time, ros battery -->
+    <include filename="$(find pr2_description)/gazebo/gazebo.urdf.xacro" />
+    <!-- materials for visualization -->
+    <include filename="$(find pr2_description)/urdf/materials.urdf.xacro" />
+    <!-- Now we can start using the macros included above to define the actual PR2 -->
+    <!-- The first use of a macro.  This one was defined in base.urdf.xacro above.
+       A macro like this will expand to a set of link and joint definitions, and to additional
+       Gazebo-related extensions (sensor plugins, etc).  The macro takes an argument, name,
+       that equals "base", and uses it to generate names for its component links and joints
+       (e.g., base_link).  The included origin block is also an argument to the macro.  By convention,
+       the origin block defines where the component is w.r.t its parent (in this case the parent
+       is the world frame). For more, see http://www.ros.org/wiki/xacro -->
+    <xacro:pr2_base_v0 name="base"/>
+    <xacro:pr2_torso_v0 name="torso_lift" parent="base_link">
+    <origin xyz="-0.05 0 0.739675" rpy="0 0 0" />
+    </xacro:pr2_torso_v0>
+    <!-- The xacro preprocesser will replace the parameters below, such as ${cal_head_x}, with
+       numerical values that were specified in common.xacro which was included above -->
+    <xacro:pr2_head_v0 name="head" parent="torso_lift_link">
+    <origin xyz="-0.01707 0.0 0.38145"
+            rpy="0.0 0.0 0.0" />
+    </xacro:pr2_head_v0>
 </robot>

Commit message: pr2 works

File: navi_model/urdf/navi.urdf.xacro (robot description, xacro)
@@ -7,25 +7,8 @@
     <!-- misc common stuff? -->
     <include filename="$(find pr2_description)/urdf/common.xacro" />
-    <!-- PR2 Arm -->
-    <include filename="$(find pr2_description)/urdf/shoulder_v0/shoulder.urdf.xacro" />
-    <include filename="$(find pr2_description)/urdf/upper_arm_v0/upper_arm.urdf.xacro" />
-    <include filename="$(find pr2_description)/urdf/forearm_v0/forearm.urdf.xacro" />
-    <!-- PR2 gripper -->
-    <include filename="$(find pr2_description)/urdf/gripper_v0/gripper.urdf.xacro" />
-    <!-- PR2 head -->
-    <include filename="$(find pr2_description)/urdf/head_v0/head.urdf.xacro" />
-    <!-- PR2 tilting laser mount -->
-    <include filename="$(find pr2_description)/urdf/tilting_laser_v0/tilting_laser.urdf.xacro" />
     <!-- PR2 torso -->
     <include filename="$(find pr2_description)/urdf/torso_v0/torso.urdf.xacro" />
     <!-- PR2 base -->
     <include filename="$(find pr2_description)/urdf/base_v0/base.urdf.xacro" />
-    <!-- Head sensors -->
-    <include filename="$(find pr2_description)/urdf/sensors/head_sensor_package.urdf.xacro" />
-    <include filename="$(find pr2_description)/urdf/sensors/kinect_prosilica_camera.urdf.xacro" />
-    <!-- Camera sensors -->
-    <include filename="$(find pr2_description)/urdf/sensors/wge100_camera.urdf.xacro" />
-    <!-- Texture projector -->
-    <include filename="$(find pr2_description)/urdf/sensors/projector_wg6802418.urdf.xacro" />
     <!-- generic simulator_gazebo plugins for starting mechanism control, ros time, ros battery -->
     <include filename="$(find pr2_description)/gazebo/gazebo.urdf.xacro" />
@@ -41,12 +24,3 @@
        is the world frame). For more, see http://www.ros.org/wiki/xacro -->
     <xacro:pr2_base_v0 name="base"/>
-    <xacro:pr2_torso_v0 name="torso_lift" parent="base_link">
-    <origin xyz="-0.05 0 0.739675" rpy="0 0 0" />
-    </xacro:pr2_torso_v0>
-    <!-- The xacro preprocesser will replace the parameters below, such as ${cal_head_x}, with
-       numerical values that were specified in common.xacro which was included above -->
-    <xacro:pr2_head_v0 name="head" parent="torso_lift_link">
-    <origin xyz="-0.01707 0.0 0.38145"
-            rpy="0.0 0.0 0.0" />
-    </xacro:pr2_head_v0>
 </robot>
