Commit message: Reverted to actual Navi model.
This reverts commit 20e43ff87cfdb0325150cc3de460ee62a0309874.

File: navi_model/urdf/navi.urdf.xacro (robot description, xacro)
@@ -1,26 +1,181 @@
 <?xml version="1.0"?>
-<robot xmlns:controller="http://playerstage.sourceforge.net/gazebo/xmlschema/#controller"
+<robot xmlns:body="http://playerstage.sourceforge.net/gazebo/xmlschema/#body"
+       xmlns:controller="http://playerstage.sourceforge.net/gazebo/xmlschema/#controller"
+       xmlns:geom="http://playerstage.sourceforge.net/gazebo/xmlschema/#geom"
        xmlns:interface="http://playerstage.sourceforge.net/gazebo/xmlschema/#interface"
+       xmlns:joint="http://playerstage.sourceforge.net/gazebo/xmlschema/#slider"
+       xmlns:sensor="http://playerstage.sourceforge.net/gazebo/xmlschema/#sensor"
        xmlns:xacro="http://ros.org/wiki/xacro"
        name="navi">
-    <!-- The following included files set up definitions of parts of the robot body -->
-    <!-- misc common stuff? -->
-    <include filename="$(find pr2_description)/urdf/common.xacro" />
-    <!-- PR2 torso -->
-    <include filename="$(find pr2_description)/urdf/torso_v0/torso.urdf.xacro" />
-    <!-- PR2 base -->
-    <include filename="$(find pr2_description)/urdf/base_v0/base.urdf.xacro" />
-    <!-- generic simulator_gazebo plugins for starting mechanism control, ros time, ros battery -->
-    <include filename="$(find pr2_description)/gazebo/gazebo.urdf.xacro" />
-    <!-- materials for visualization -->
-    <include filename="$(find pr2_description)/urdf/materials.urdf.xacro" />
-    <!-- Now we can start using the macros included above to define the actual PR2 -->
-    <!-- The first use of a macro.  This one was defined in base.urdf.xacro above.
-       A macro like this will expand to a set of link and joint definitions, and to additional
-       Gazebo-related extensions (sensor plugins, etc).  The macro takes an argument, name,
-       that equals "base", and uses it to generate names for its component links and joints
-       (e.g., base_link).  The included origin block is also an argument to the macro.  By convention,
-       the origin block defines where the component is w.r.t its parent (in this case the parent
-       is the world frame). For more, see http://www.ros.org/wiki/xacro -->
-    <xacro:pr2_base_v0 name="base"/>
+    <xacro:property name="EPS" value="0.000001"/>
+    <xacro:property name="PI" value="3.1415926535897931"/>
+    <xacro:property name="robot_weight" value="90.0"/>
+    <xacro:property name="wheel_radius" value="0.127"/>
+    <xacro:property name="wheel_thickness" value="0.0762"/>
+    <xacro:property name="wheel_separation" value="0.70386"/>
+    <xacro:property name="wheel_mass" value="3.175"/>
+    <xacro:property name="wheel_torque" value="10"/>
+    <xacro:property name="robot_clearance" value="0.3937"/>
+    <xacro:property name="caster_radius" value="0.1143"/>
+    <xacro:property name="caster_thickness" value="0.0508"/>
+    <xacro:property name="caster_separation" value="0.53388"/>
+    <xacro:property name="caster_clearance" value="0.254"/>
+    <xacro:property name="caster_mass" value="2.268"/>
+    <xacro:property name="caster_offset_height" value="0.1524"/>
+    <xacro:property name="caster_offset_axis" value="0.0889"/>
+    <xacro:property name="mesh_offset" value="-0.60 0.300 -0.50"/>
+    <xacro:macro name="weightless">
+        <inertial>
+            <mass value="${EPS}"/>
+            <inertia ixx="${EPS}" ixy="0"      ixz="0"
+                                  iyy="${EPS}" iyz="0"
+                                               izz="${EPS}"/>
+        </inertial>
+    </xacro:macro>
+    <xacro:macro name="chassis">
+        <link name="base_link">
+            <inertial>
+                <mass value="1.0"/>
+                <inertia ixx="1.0" ixy="0.0"   ixz="0.0"
+                                   iyy="100.0" iyz="0.0"
+                                               izz="1.0" />
+            </inertial>
+            <visual>
+                <origin xyz="${mesh_offset}" rpy="${PI/2} 0 0"/>
+                <geometry>
+                    <mesh filename="package://navi_model/meshes/frame.stl" scale="0.001 0.001 0.001"/>
+                </geometry>
+            </visual>
+            <collision>
+                <geometry>
+                    <box size="0.9 0.8 0.3"/>
+                </geometry>
+            </collision>
+        </link>
+        <gazebo reference="base_link">
+            <material>Gazebo/Blue</material>
+        </gazebo>
+        <joint name="base_link_joint" type="fixed">
+            <parent link="base_link"/>
+            <child link="base_footprint"/>
+            <origin xyz="0 0 ${-robot_clearance - wheel_radius}"/>
+        </joint>
+        <link name="base_footprint">
+            <xacro:weightless/>
+        </link>
+    </xacro:macro>
+    <xacro:macro name="wheel" params="side sign">
+        <joint name="wheel_${side}_joint" type="continuous">
+            <parent link="base_link"/>
+            <child link="wheel_${side}_link"/>
+            <origin xyz="0 ${sign*wheel_separation/2} ${-robot_clearance}" rpy="${PI/2} 0 0"/>
+            <axis xyz="0 0 1"/>
+        </joint>
+        <link name="wheel_${side}_link">
+            <inertial>
+                <mass value="${wheel_mass}"/>
+                <inertia ixx="${wheel_mass*(3*wheel_radius*wheel_radius + wheel_thickness*wheel_thickness)}" ixy="0.0" ixz="0.0"
+                         iyy="${wheel_mass*(3*wheel_radius*wheel_radius + wheel_thickness*wheel_thickness)}" iyz="0.0"
+                         izz="${wheel_mass*wheel_radius*wheel_radius/2}"/>
+            </inertial>
+            <visual>
+                <geometry>
+                    <cylinder radius="${wheel_radius}" length="${wheel_thickness}"/>
+                </geometry>
+            </visual>
+            <collision>
+                <geometry>
+                    <cylinder radius="${wheel_radius}" length="${wheel_thickness}"/>
+                </geometry>
+            </collision>
+        </link>
+        <gazebo reference="wheel_${side}_link">
+            <material>Gazebo/Red</material>
+        </gazebo>
+    </xacro:macro>
+    <xacro:macro name="caster">
+        <joint name="caster_pivot_joint" type="continuous">
+            <parent link="base_link"/>
+            <child link="caster_pivot_link"/>
+            <origin xyz="${-caster_separation} 0 ${-caster_clearance)}"
+                    rpy="${PI/2} 0 0"/>
+            <axis xyz="0 1 0"/>
+        </joint>
+        <link name="caster_pivot_link">
+            <inertial>
+                <mass value="${caster_mass}"/>
+                <inertia ixx="${EPS}" ixy="0"      ixz="0"
+                                      iyy="${EPS}" iyz="0"
+                                                   izz="${EPS}"/>
+            </inertial>
+        </link>
+        <!-- TODO: Why can't I make this continuous? -->
+        <joint name="caster_joint" type="fixed">
+            <parent link="caster_pivot_link"/>
+            <child link="caster_link"/>
+            <origin xyz="${-caster_offset_axis} ${-caster_offset_height} 0"/>
+            <axis xyz="0 0 1"/>
+        </joint>
+        <link name="caster_link">
+            <inertial>
+                <mass value="${caster_mass}"/>
+                <inertia ixx="${caster_mass*(3*caster_radius*caster_radius + caster_thickness*caster_thickness)}" ixy="0.0" ixz="0.0"
+                         iyy="${caster_mass*(3*caster_radius*caster_radius + caster_thickness*caster_thickness)}" iyz="0.0"
+                         izz="${caster_mass*caster_radius*caster_radius/2}"/>
+            </inertial>
+            <visual>
+                <inertia ixx="${wheel_mass*(3*wheel_radius*wheel_radius + wheel_thickness*wheel_thickness)}" ixy="0.0" ixz="0.0"
+                         iyy="${wheel_mass*(3*wheel_radius*wheel_radius + wheel_thickness*wheel_thickness)}" iyz="0.0"
+                         izz="${wheel_mass*wheel_radius*wheel_radius/2}"/>
+                <geometry>
+                    <cylinder radius="${caster_radius}" length="${caster_thickness}"/>
+                </geometry>
+            </visual>
+            <collision>
+                <geometry>
+                    <cylinder radius="${caster_radius}" length="${caster_thickness}"/>
+                </geometry>
+            </collision>
+        </link>
+        <gazebo reference="caster_link">
+            <material>Gazebo/Red</material>
+        </gazebo>
+    </xacro:macro>
+    <xacro:macro name="gazebo_drive">
+        <gazebo>
+            <controller:diffdrive_plugin name="differential_drive_controller" plugin="libdiffdrive_plugin.so">
+                <alwaysOn>true</alwaysOn>
+                <update>100</update>
+                <updateRate>100.0</updateRate>
+                <torque>${wheel_torque}</torque>
+                <wheelSeparation>${wheel_separation}</wheelSeparation>
+                <wheelDiameter>${wheel_radius*2}</wheelDiameter>
+                <robotNamespace>/</robotNamespace>
+                <topicName>drive/cmd_vel</topicName>
+                <leftJoint>wheel_left_joint</leftJoint>
+                <rightJoint>wheel_right_joint</rightJoint>
+                <interface:position name="drive_iface"/>
+            </controller:diffdrive_plugin>
+        </gazebo>
+    </xacro:macro>
+    <xacro:macro name="gazebo_localization">
+        <gazebo>
+            <controller:gazebo_ros_p3d name="gps_controller" plugin="libgazebo_ros_p3d.so">
+                <alwaysOn>true</alwaysOn>
+                <updateRate>60</updateRate>
+                <bodyName>base_link</bodyName>
+                <topicName>ground_truth</topicName>
+                <gaussianNoise>0.0</gaussianNoise>
+                <frameName>/map</frameName>
+                <interface:position name="gps_iface"/>
+            </controller:gazebo_ros_p3d>
+            <canonicalBody>base_link</canonicalBody>
+        </gazebo>
+    </xacro:macro>
+    <xacro:chassis/>
+    <xacro:wheel sign="-1" side="left"/>
+    <xacro:wheel sign="+1" side="right"/>
+    <xacro:caster/>
+    <xacro:gazebo_drive/>
+    <xacro:gazebo_localization/>
 </robot>

Commit message: collision model is correct

File: navi_model/urdf/navi.urdf.xacro (robot description, xacro)
@@ -34,4 +34,12 @@
     </xacro:macro>
     <xacro:macro name="chassis">
+        <link name="base_footprint">
+            <xacro:weightless/>
+        </link>
+        <joint name="base_link_joint" type="fixed">
+            <parent link="base_footprint"/>
+            <child link="base_link"/>
+            <origin xyz="0 0 ${robot_clearance + wheel_radius}"/>
+        </joint>
         <link name="base_link">
             <inertial>
@@ -56,12 +64,4 @@
             <material>Gazebo/Blue</material>
         </gazebo>
-        <joint name="base_link_joint" type="fixed">
-            <parent link="base_link"/>
-            <child link="base_footprint"/>
-            <origin xyz="0 0 ${-robot_clearance - wheel_radius}"/>
-        </joint>
-        <link name="base_footprint">
-            <xacro:weightless/>
-        </link>
     </xacro:macro>
     <xacro:macro name="wheel" params="side sign">

Commit message: added grass simulation

File: navi_model/urdf/navi.urdf.xacro (robot description, xacro)
@@ -24,5 +24,5 @@
     <xacro:property name="caster_offset_height" value="0.1524"/>
     <xacro:property name="caster_offset_axis" value="0.0889"/>
-    <xacro:property name="mesh_offset" value="-0.60 0.300 -0.50"/>
+    <xacro:property name="mesh_offset" value="0 0 0"/>
     <xacro:macro name="weightless">
         <inertial>
@@ -50,5 +50,5 @@
             </inertial>
             <visual>
-                <origin xyz="${mesh_offset}" rpy="${PI/2} 0 0"/>
+                <origin xyz="0 0.52 0.07" rpy="${PI/2} 0 0"/>
                 <geometry>
                     <mesh filename="package://navi_model/meshes/frame.stl" scale="0.001 0.001 0.001"/>

Commit message: split urdf into separate files

File: navi_model/urdf/navi.urdf.xacro (robot description, xacro)
@@ -28,152 +28,10 @@
         <inertial>
             <mass value="${EPS}"/>
-            <inertia ixx="${EPS}" ixy="0"      ixz="0"
-                                  iyy="${EPS}" iyz="0"
-                                               izz="${EPS}"/>
+            <inertia ixx="${EPS}" ixy="0" ixz="0" iyy="${EPS}" iyz="0" izz="${EPS}"/>
         </inertial>
     </xacro:macro>
-    <xacro:macro name="chassis">
-        <link name="base_footprint">
-            <xacro:weightless/>
-        </link>
-        <joint name="base_link_joint" type="fixed">
-            <parent link="base_footprint"/>
-            <child link="base_link"/>
-            <origin xyz="0 0 ${robot_clearance + wheel_radius}"/>
-        </joint>
-        <link name="base_link">
-            <inertial>
-                <mass value="1.0"/>
-                <inertia ixx="1.0" ixy="0.0"   ixz="0.0"
-                                   iyy="100.0" iyz="0.0"
-                                               izz="1.0" />
-            </inertial>
-            <visual>
-                <origin xyz="0 0.52 0.07" rpy="${PI/2} 0 0"/>
-                <geometry>
-                    <mesh filename="package://navi_model/meshes/frame.stl" scale="0.001 0.001 0.001"/>
-                </geometry>
-            </visual>
-            <collision>
-                <geometry>
-                    <box size="0.9 0.8 0.3"/>
-                </geometry>
-            </collision>
-        </link>
-        <gazebo reference="base_link">
-            <material>Gazebo/Blue</material>
-        </gazebo>
-    </xacro:macro>
-    <xacro:macro name="wheel" params="side sign">
-        <joint name="wheel_${side}_joint" type="continuous">
-            <parent link="base_link"/>
-            <child link="wheel_${side}_link"/>
-            <origin xyz="0 ${sign*wheel_separation/2} ${-robot_clearance}" rpy="${PI/2} 0 0"/>
-            <axis xyz="0 0 1"/>
-        </joint>
-        <link name="wheel_${side}_link">
-            <inertial>
-                <mass value="${wheel_mass}"/>
-                <inertia ixx="${wheel_mass*(3*wheel_radius*wheel_radius + wheel_thickness*wheel_thickness)}" ixy="0.0" ixz="0.0"
-                         iyy="${wheel_mass*(3*wheel_radius*wheel_radius + wheel_thickness*wheel_thickness)}" iyz="0.0"
-                         izz="${wheel_mass*wheel_radius*wheel_radius/2}"/>
-            </inertial>
-            <visual>
-                <geometry>
-                    <cylinder radius="${wheel_radius}" length="${wheel_thickness}"/>
-                </geometry>
-            </visual>
-            <collision>
-                <geometry>
-                    <cylinder radius="${wheel_radius}" length="${wheel_thickness}"/>
-                </geometry>
-            </collision>
-        </link>
-        <gazebo reference="wheel_${side}_link">
-            <material>Gazebo/Red</material>
-        </gazebo>
-    </xacro:macro>
-    <xacro:macro name="caster">
-        <joint name="caster_pivot_joint" type="continuous">
-            <parent link="base_link"/>
-            <child link="caster_pivot_link"/>
-            <origin xyz="${-caster_separation} 0 ${-caster_clearance)}"
-                    rpy="${PI/2} 0 0"/>
-            <axis xyz="0 1 0"/>
-        </joint>
-        <link name="caster_pivot_link">
-            <inertial>
-                <mass value="${caster_mass}"/>
-                <inertia ixx="${EPS}" ixy="0"      ixz="0"
-                                      iyy="${EPS}" iyz="0"
-                                                   izz="${EPS}"/>
-            </inertial>
-        </link>
-        <!-- TODO: Why can't I make this continuous? -->
-        <joint name="caster_joint" type="fixed">
-            <parent link="caster_pivot_link"/>
-            <child link="caster_link"/>
-            <origin xyz="${-caster_offset_axis} ${-caster_offset_height} 0"/>
-            <axis xyz="0 0 1"/>
-        </joint>
-        <link name="caster_link">
-            <inertial>
-                <mass value="${caster_mass}"/>
-                <inertia ixx="${caster_mass*(3*caster_radius*caster_radius + caster_thickness*caster_thickness)}" ixy="0.0" ixz="0.0"
-                         iyy="${caster_mass*(3*caster_radius*caster_radius + caster_thickness*caster_thickness)}" iyz="0.0"
-                         izz="${caster_mass*caster_radius*caster_radius/2}"/>
-            </inertial>
-            <visual>
-                <inertia ixx="${wheel_mass*(3*wheel_radius*wheel_radius + wheel_thickness*wheel_thickness)}" ixy="0.0" ixz="0.0"
-                         iyy="${wheel_mass*(3*wheel_radius*wheel_radius + wheel_thickness*wheel_thickness)}" iyz="0.0"
-                         izz="${wheel_mass*wheel_radius*wheel_radius/2}"/>
-                <geometry>
-                    <cylinder radius="${caster_radius}" length="${caster_thickness}"/>
-                </geometry>
-            </visual>
-            <collision>
-                <geometry>
-                    <cylinder radius="${caster_radius}" length="${caster_thickness}"/>
-                </geometry>
-            </collision>
-        </link>
-        <gazebo reference="caster_link">
-            <material>Gazebo/Red</material>
-        </gazebo>
-    </xacro:macro>
-    <xacro:macro name="gazebo_drive">
-        <gazebo>
-            <controller:diffdrive_plugin name="differential_drive_controller" plugin="libdiffdrive_plugin.so">
-                <alwaysOn>true</alwaysOn>
-                <updateRate>50.0</updateRate>
-                <torque>${wheel_torque}</torque>
-                <leftJoint>wheel_left_joint</leftJoint>
-                <rightJoint>wheel_right_joint</rightJoint>
-                <wheelSeparation>${wheel_separation}</wheelSeparation>
-                <wheelDiameter>${wheel_radius*2}</wheelDiameter>
-                <robotNamespace>/</robotNamespace>
-                <baseFrame>base_footprint</baseFrame>
-                <odomFrame>odom</odomFrame>
-                <twistTopicName>drive/cmd_vel</twistTopicName>
-                <odomTopicName>drive/odom</odomTopicName>
-                <alpha>0.05</alpha>
-                <interface:position name="drive_iface"/>
-            </controller:diffdrive_plugin>
-        </gazebo>
-    </xacro:macro>
-    <xacro:macro name="gazebo_localization">
-        <gazebo>
-            <controller:gazebo_ros_p3d name="gps_controller" plugin="libgazebo_ros_p3d.so">
-                <alwaysOn>true</alwaysOn>
-                <updateRate>60</updateRate>
-                <bodyName>base_footprint</bodyName>
-                <topicName>/ground_truth</topicName>
-                <gaussianNoise>0.0</gaussianNoise>
-                <frameName>/map</frameName>
-                <interface:position name="gps_iface"/>
-            </controller:gazebo_ros_p3d>
-            <canonicalBody>base_footprint</canonicalBody>
-        </gazebo>
-    </xacro:macro>
+    <include filename="$(find navi_model)/urdf/chassis.urdf.xacro"/>
+    <include filename="$(find navi_model)/urdf/wheels.urdf.xacro"/>
+    <include filename="$(find navi_model)/urdf/gazebo.urdf.xacro"/>
     <xacro:chassis/>
     <xacro:wheel sign="-1" side="left"/>

Commit message: added simulated cameras

File: navi_model/urdf/navi.urdf.xacro (robot description, xacro)
@@ -25,4 +25,12 @@
     <xacro:property name="caster_offset_axis" value="0.0889"/>
     <xacro:property name="mesh_offset" value="0 0 0"/>
+    <xacro:property name="gps_offset" value="-0.18941 0 0.76387"/>
+    <xacro:property name="laser_offset" value="0.02927 0 0.46714"/>
+    <xacro:property name="camera_x" value="-0.09717"/>
+    <xacro:property name="camera_y" value="0.24582"/>
+    <xacro:property name="camera_z" value="0.75734"/>
+    <xacro:property name="camera_roll"  value="0"/>
+    <xacro:property name="camera_pitch" value="0.177150919"/>
+    <xacro:property name="camera_yaw"   value="0.174532925"/>
     <xacro:macro name="weightless">
         <inertial>
@@ -31,11 +39,26 @@
         </inertial>
     </xacro:macro>
+    <xacro:macro name="frame" params="parent child xyz rpy">
+        <joint name="${child}_joint" type="fixed">
+            <parent link="${parent}"/>
+            <child link="${child}"/>
+            <origin xyz="${xyz}" rpy="${rpy}"/>
+        </joint>
+        <link name="${child}">
+            <xacro:weightless/>
+        </link>
+    </xacro:macro>
+    <include filename="$(find navi_model)/urdf/cameras.urdf.xacro"/>
     <include filename="$(find navi_model)/urdf/chassis.urdf.xacro"/>
+    <include filename="$(find navi_model)/urdf/gazebo.urdf.xacro"/>
     <include filename="$(find navi_model)/urdf/wheels.urdf.xacro"/>
-    <include filename="$(find navi_model)/urdf/gazebo.urdf.xacro"/>
     <xacro:chassis/>
-    <xacro:wheel sign="-1" side="left"/>
-    <xacro:wheel sign="+1" side="right"/>
+    <xacro:wheel sign="+1" side="left"/>
+    <xacro:wheel sign="-1" side="right"/>
     <xacro:caster/>
+    <xacro:camera sign="+1" side="left"/>
+    <xacro:camera sign="-1" side="right"/>
+    <xacro:frame parent="base_link" child="gps" xyz="${gps_offset}" rpy="0 0 0"/>
+    <xacro:frame parent="base_link" child="laser" xyz="${laser_offset}" rpy="0 0 0"/>
     <xacro:gazebo_drive/>
     <xacro:gazebo_localization/>
