Commit message: caster is only semi-broken

File: navi_model/urdf/navi.urdf.xacro (robot description, xacro)
@@ -14,7 +14,9 @@
     <xacro:property name="wheel_radius" value="0.127"/>
     <xacro:property name="wheel_thickness" value="0.0762"/>
-    <xacro:property name="wheel_separation" value="0.70386"/>
+    <xacro:property name="wheel_separation" value="0.70354"/>
     <xacro:property name="wheel_mass" value="3.175"/>
     <xacro:property name="wheel_torque" value="10"/>
+    <xacro:property name="caster_pivot_offset" value="-0.53388 0  0.10833"/>
+    <xacro:property name="caster_wheel_offset" value="-0.07620 0 -0.12103"/>
     <xacro:property name="caster_radius" value="0.1143"/>
     <xacro:property name="caster_thickness" value="0.0508"/>
@@ -24,5 +26,4 @@
     <xacro:property name="caster_offset_height" value="0.1524"/>
     <xacro:property name="caster_offset_axis" value="0.0889"/>
-    <xacro:property name="mesh_offset" value="0 0 0"/>
     <xacro:property name="gps_offset" value="-0.18941 0 0.76387"/>
     <xacro:property name="laser_offset" value="0.02927 0 0.46714"/>
@@ -50,14 +51,10 @@
     <xacro:wheel sign="+1" side="left"/>
     <xacro:wheel sign="-1" side="right"/>
-    <!--
     <xacro:caster/>
-    -->
     <xacro:camera sign="+1" side="left"/>
     <xacro:camera sign="-1" side="right"/>
     <xacro:frame parent="base_link" child="gps" xyz="${gps_offset}" rpy="0 0 0"/>
     <xacro:frame parent="base_link" child="laser" xyz="${laser_offset}" rpy="0 0 0"/>
-    <!--
     <xacro:gazebo_drive/>
     <xacro:gazebo_localization/>
-    -->
 </robot>

File: navi_model/urdf/wheels.urdf.xacro (robot description, xacro)
@@ -40,7 +40,6 @@
             <parent link="base_link"/>
             <child link="caster_pivot_link"/>
-            <origin xyz="${-caster_separation} 0 ${-caster_clearance)}"
-                    rpy="${PI/2} 0 0"/>
-            <axis xyz="0 1 0"/>
+            <origin xyz="${caster_pivot_offset}"/>
+            <axis xyz="0 0 1"/>
         </joint>
         <link name="caster_pivot_link">
@@ -55,5 +54,5 @@
             <parent link="caster_pivot_link"/>
             <child link="caster_link"/>
-            <origin xyz="${-caster_offset_axis} ${-caster_offset_height} 0"/>
+            <origin xyz="${caster_wheel_offset}" rpy="${PI/2} 0 0"/>
             <axis xyz="0 0 1"/>
         </joint>
