Commit message: fixed model in rviz and gazebo

File: navi_model/urdf/chassis.urdf.xacro (robot description, xacro)
@@ -24,14 +24,31 @@
             </inertial>
             <visual>
-                <origin xyz="0 0 ${2*wheel_radius}" rpy="0 0 0"/>
+                <origin xyz="0 0 ${3*wheel_radius}" rpy="0 0 0"/>
                 <geometry>
-                    <box size="0.9 0.8 0.3"/>
-                    <!--<mesh filename="package://navi_model/meshes/frame.stl" scale="0.001 0.001 0.001"/>-->
+                    <box size="${EPS} ${EPS} ${EPS}"/>
                 </geometry>
             </visual>
             <collision>
-                <origin xyz="0 0 ${4*wheel_radius}" rpy="0 0 0"/>
+                <origin xyz="0 0 ${3*wheel_radius}" rpy="0 0 0"/>
                 <geometry>
-                    <box size="0.9 0.8 0.3"/>
+                    <box size="${EPS} ${EPS} ${EPS}"/>
+                </geometry>
+            </collision>
+        </link>
+        <joint name="visual_joint" type="fixed">
+            <parent link="base_link"/>
+            <child link="visual_link"/>
+            <origin xyz="0 0 0" rpy="${PI/2} 0 0"/>
+        </joint>
+        <link name="visual_link">
+            <xacro:weightless/>
+            <visual>
+                <geometry>
+                    <mesh filename="package://navi_model/meshes/frame.stl" scale="0.001 0.001 0.001"/>
+                </geometry>
+            </visual>
+            <collision>
+                <geometry>
+                    <mesh filename="package://navi_model/meshes/frame.stl" scale="0.001 0.001 0.001"/>
                 </geometry>
             </collision>

Commit message: changed colors in rviz

File: navi_model/urdf/chassis.urdf.xacro (robot description, xacro)
@@ -36,10 +36,10 @@
             </collision>
         </link>
-        <joint name="visual_joint" type="fixed">
+        <joint name="base_visual_joint" type="fixed">
             <parent link="base_link"/>
-            <child link="visual_link"/>
+            <child link="base_visual"/>
             <origin xyz="0 0 0" rpy="${PI/2} 0 0"/>
         </joint>
-        <link name="visual_link">
+        <link name="base_visual">
             <xacro:weightless/>
             <visual>
@@ -47,4 +47,5 @@
                     <mesh filename="package://navi_model/meshes/frame.stl" scale="0.001 0.001 0.001"/>
                 </geometry>
+                <material name="Blue"/>
             </visual>
             <collision>
@@ -54,5 +55,5 @@
             </collision>
         </link>
-        <gazebo reference="base_link">
+        <gazebo reference="base_visual">
             <material>Gazebo/Blue</material>
         </gazebo>

File: navi_model/urdf/materials.urdf.xacro (robot description, xacro)
@@ -1,12 +1,15 @@
 <?xml version="1.0"?>
 <robot>
-    <material name="red">
-        <color rgba="1 0 0 1"/>
+    <material name="Red">
+        <color rgba="0.8 0.0 0.0 1.0"/>
     </material>
-    <material name="green">
-        <color rgba="0 1 0 1"/>
+    <material name="Green">
+        <color rgba="0.0 0.8 0.0 1.0"/>
     </material>
-    <material name="blue">
-        <color rgba="0 0 1 1"/>
+    <material name="Blue">
+        <color rgba="0.0 0.0 0.8 1.0"/>
+    </material>
+    <material name="Grey">
+        <color rgba="0.7 0.7 0.7 1.0"/>
     </material>
 </robot>

File: navi_model/urdf/navi.urdf.xacro (robot description, xacro)
@@ -44,4 +44,5 @@
         </link>
     </xacro:macro>
+    <include filename="$(find navi_model)/urdf/materials.urdf.xacro"/>
     <include filename="$(find navi_model)/urdf/cameras.urdf.xacro"/>
     <include filename="$(find navi_model)/urdf/chassis.urdf.xacro"/>

File: navi_model/urdf/wheels.urdf.xacro (robot description, xacro)
@@ -25,4 +25,5 @@
                     <cylinder radius="${wheel_radius}" length="${wheel_thickness}"/>
                 </geometry>
+                <material name="Grey"/>
             </visual>
             <collision>
@@ -33,5 +34,5 @@
         </link>
         <gazebo reference="wheel_${side}_link">
-            <material>Gazebo/Red</material>
+            <material>Gazebo/Grey</material>
         </gazebo>
     </xacro:macro>
@@ -71,4 +72,5 @@
                     <cylinder radius="${caster_radius}" length="${caster_thickness}"/>
                 </geometry>
+                <material name="Grey"/>
             </visual>
             <collision>
@@ -79,5 +81,5 @@
         </link>
         <gazebo reference="caster_link">
-            <material>Gazebo/Red</material>
+            <material>Gazebo/Grey</material>
         </gazebo>
     </xacro:macro>

Commit message: split up gazebo plugins

File: navi_model/urdf/chassis.urdf.xacro (robot description, xacro)
@@ -58,4 +58,22 @@
             <material>Gazebo/Blue</material>
         </gazebo>
+        <gazebo>
+            <controller:diffdrive_plugin name="differential_drive_controller" plugin="libdiffdrive_plugin.so">
+                <alwaysOn>true</alwaysOn>
+                <updateRate>50.0</updateRate>
+                <torque>${wheel_torque}</torque>
+                <leftJoint>wheel_left_joint</leftJoint>
+                <rightJoint>wheel_right_joint</rightJoint>
+                <wheelSeparation>${wheel_separation}</wheelSeparation>
+                <wheelDiameter>${2*wheel_radius}</wheelDiameter>
+                <robotNamespace>/</robotNamespace>
+                <baseFrame>base_footprint</baseFrame>
+                <odomFrame>odom</odomFrame>
+                <twistTopicName>drive/cmd_vel</twistTopicName>
+                <odomTopicName>drive/odom</odomTopicName>
+                <alpha>0.05</alpha>
+                <interface:position name="drive_iface"/>
+            </controller:diffdrive_plugin>
+        </gazebo>
     </xacro:macro>
 </robot>

File: navi_model/urdf/gps.urdf.xacro (robot description, xacro)
@@ -7,25 +7,6 @@
        xmlns:sensor="http://playerstage.sourceforge.net/gazebo/xmlschema/#sensor"
        xmlns:xacro="http://ros.org/wiki/xacro">
-    <xacro:macro name="gazebo_drive">
-        <gazebo>
-            <controller:diffdrive_plugin name="differential_drive_controller" plugin="libdiffdrive_plugin.so">
-                <alwaysOn>true</alwaysOn>
-                <updateRate>50.0</updateRate>
-                <torque>${wheel_torque}</torque>
-                <leftJoint>wheel_left_joint</leftJoint>
-                <rightJoint>wheel_right_joint</rightJoint>
-                <wheelSeparation>${wheel_separation}</wheelSeparation>
-                <wheelDiameter>${2*wheel_radius}</wheelDiameter>
-                <robotNamespace>/</robotNamespace>
-                <baseFrame>base_footprint</baseFrame>
-                <odomFrame>odom</odomFrame>
-                <twistTopicName>drive/cmd_vel</twistTopicName>
-                <odomTopicName>drive/odom</odomTopicName>
-                <alpha>0.05</alpha>
-                <interface:position name="drive_iface"/>
-            </controller:diffdrive_plugin>
-        </gazebo>
-    </xacro:macro>
-    <xacro:macro name="gazebo_localization">
+    <xacro:macro name="gps">
+        <xacro:frame parent="base_link" child="gps" xyz="${gps_offset}" rpy="0 0 0"/>
         <gazebo>
             <controller:gazebo_ros_p3d name="gps_controller" plugin="libgazebo_ros_p3d.so">

File: navi_model/urdf/navi.urdf.xacro (robot description, xacro)
@@ -55,8 +55,6 @@
     <xacro:caster/>
     <xacro:laser/>
+    <xacro:gps/>
     <xacro:camera sign="+1" side="left"/>
     <xacro:camera sign="-1" side="right"/>
-    <xacro:frame parent="base_link" child="gps" xyz="${gps_offset}" rpy="0 0 0"/>
-    <xacro:gazebo_drive/>
-    <xacro:gazebo_localization/>
 </robot>
