Commit message: added camera pitch roll and yaw

File: navi_model/urdf/cameras.urdf.xacro (robot description, xacro)
@@ -11,9 +11,12 @@
     <xacro:property name="camera_y" value="0.24592"/>
     <xacro:property name="camera_z" value="0.75734"/>
+    <xacro:property name="camera_roll" value="0.17715"/>
+    <xacro:property name="camera_yaw"  value="0.17453"/>
     <xacro:macro name="camera" params="side sign">
         <joint name="camera_${side}_joint" type="fixed">
             <parent link="base_link"/>
             <child link="camera_${side}_link"/>
-            <origin xyz="${camera_x} ${sign*camera_y} ${camera_z}" rpy="${PI/2} ${PI} ${PI/2}"/>
+            <origin xyz="${camera_x} ${sign*camera_y} ${camera_z}"
+                    rpy="${PI/2 - camera_roll} ${PI} ${PI/2 + sign*camera_yaw}"/>
             <!-- TODO: This rotation is wrong. -->
             <axis xyz="0 0 0"/>

Commit message: added cameras to gazebo simulation; pose wrong

File: navi_model/urdf/cameras.urdf.xacro (robot description, xacro)
@@ -13,4 +13,8 @@
     <xacro:property name="camera_roll" value="0.17715"/>
     <xacro:property name="camera_yaw"  value="0.17453"/>
+    <xacro:property name="camera_fps" value="20"/>
+    <xacro:property name="camera_resx" value="640"/>
+    <xacro:property name="camera_resy" value="480"/>
+    <xacro:property name="camera_hfov" value="1.39626"/> <!-- 80 degrees -->
     <xacro:macro name="camera" params="side sign">
         <joint name="camera_${side}_joint" type="fixed">
@@ -19,9 +23,43 @@
             <origin xyz="${camera_x} ${sign*camera_y} ${camera_z}"
                     rpy="${PI/2 - camera_roll} ${PI} ${PI/2 + sign*camera_yaw}"/>
+            <axis xyz="0 0 0"/>
+            <anchor xyz="0 0 0"/>
+        </joint>
+        <link name="camera_${side}_link"/>
+        <joint name="camera_${side}_gazebo_joint" type="fixed">
+            <parent link="camera_${side}_link"/>
+            <child link="camera_${side}_gazebo_link"/>
+            <origin xyz="0 0 0" rpy="0 0 0"/>
             <!-- TODO: This rotation is wrong. -->
             <axis xyz="0 0 0"/>
             <anchor xyz="0 0 0"/>
         </joint>
-        <link name="camera_${side}_link"/>
+        <link name="camera_${side}_gazebo_link"/>
+        <gazebo>
+            <sensor:camera name="camera_${side}_sensor">
+                <imageSize>${camera_resx} ${camera_resy}</imageSize>
+                <imageFormat>R8G8B8</imageFormat>
+                <hfov>${camera_hfov}</hfov>
+                <nearClip>0.1</nearClip>
+                <farClip>100</farClip>
+                <updateRate>${camera_fps}</updateRate>
+                <controller:gazebo_ros_camera name="camera_${side}_controller" plugin="libgazebo_ros_camera.so">
+                    <alwaysOn>true</alwaysOn>
+                    <updateRate>${camera_fps}</updateRate>
+                    <imageTopicName>camera/${side}/image_raw</imageTopicName>
+                    <cameraInfoTopicName>camera/${side}/camera_info</cameraInfoTopicName>
+                    <frameName>/camera_${side}_link</frameName>
+                    <CxPrime>${(camera_resx + 1)/2}</CxPrime>
+                    <Cx>${(camera_resx+1)/2}</Cx>
+                    <Cy>${(camera_resy+1)/2}</Cy>
+                    <distortion_k1>0.00000001</distortion_k1>
+                    <distortion_k2>0.00000001</distortion_k2>
+                    <distortion_k3>0.00000001</distortion_k3>
+                    <distortion_t1>0.00000001</distortion_t1>
+                    <distortion_t2>0.00000001</distortion_t2>
+                    <interface:camera name="camera_${side}_iface" />
+                </controller:gazebo_ros_camera>
+            </sensor:camera>
+        </gazebo>
     </xacro:macro>
 </robot>

Commit message: added dummy inertia to sensors for Gazebo

File: navi_model/urdf/cameras.urdf.xacro (robot description, xacro)
@@ -6,6 +6,5 @@
        xmlns:joint="http://playerstage.sourceforge.net/gazebo/xmlschema/#slider"
        xmlns:sensor="http://playerstage.sourceforge.net/gazebo/xmlschema/#sensor"
-       xmlns:xacro="http://ros.org/wiki/xacro"
-       name="navi">
+       xmlns:xacro="http://ros.org/wiki/xacro">
     <xacro:property name="camera_x" value="-0.09170"/>
     <xacro:property name="camera_y" value="0.24592"/>
@@ -26,5 +25,7 @@
             <anchor xyz="0 0 0"/>
         </joint>
-        <link name="camera_${side}_link"/>
+        <link name="camera_${side}_link">
+            <xacro:weightless/>
+        </link>
         <joint name="camera_${side}_gazebo_joint" type="fixed">
             <parent link="camera_${side}_link"/>
@@ -35,5 +36,8 @@
             <anchor xyz="0 0 0"/>
         </joint>
-        <link name="camera_${side}_gazebo_link"/>
+        <link name="camera_${side}_gazebo_link">
+            <xacro:weightless/>
+        </link>
+        <!--
         <gazebo>
             <sensor:camera name="camera_${side}_sensor">
@@ -62,4 +66,5 @@
             </sensor:camera>
         </gazebo>
+        -->
     </xacro:macro>
 </robot>

File: navi_model/urdf/gps.urdf.xacro (robot description, xacro)
@@ -17,5 +17,7 @@
             <anchor xyz="0 0 0"/>
         </joint>
-        <link name="gps_link"/>
+        <link name="gps_link">
+            <xacro:weightless/>
+        </link>
         <gazebo>
             <canonicalBody>gps_link</canonicalBody>

File: navi_model/urdf/laser.urdf.xacro (robot description, xacro)
@@ -17,5 +17,7 @@
             <anchor xyz="0 0 0"/>
         </joint>
-        <link name="laser_link"/>
+        <link name="laser_link">
+            <xacro:weightless/>
+        </link>
         <gazebo reference="base_laser_link">
             <sensor:ray name="laser">

File: navi_model/urdf/navi.urdf.xacro (robot description, xacro)
@@ -9,4 +9,13 @@
        name="navi">
     <xacro:property name="PI" value="3.1415926535897931"/>
+    <xacro:property name="EPS" value="0.000001"/>
+    <xacro:macro name="weightless">
+        <inertial>
+            <mass value="${EPS}"/>
+            <inertia ixx="${EPS}" ixy="0.000"  ixz="0.000"
+                                  iyy="${EPS}" iyz="0.000"
+                                               izz="${EPS}"/>
+        </inertial>
+    </xacro:macro>
     <xacro:property name="robot_width"  value="0.850"/>
     <xacro:property name="robot_length" value="1.350"/>

File: navi_model/urdf/navi_robot.urdf.xacro (robot description, xacro)
@@ -42,4 +42,6 @@
         <anchor xyz="0 0 0"/>
     </joint>
-    <link name="base_footprint"/>
+    <link name="base_footprint">
+        <xacro:weightless/>
+    </link>
 </robot>

Commit message: cameras "work", but don't generate an image

File: navi_model/urdf/cameras.urdf.xacro (robot description, xacro)
@@ -12,5 +12,5 @@
     <xacro:property name="camera_roll" value="0.17715"/>
     <xacro:property name="camera_yaw"  value="0.17453"/>
-    <xacro:property name="camera_fps" value="20"/>
+    <xacro:property name="camera_fps" value="10"/>
     <xacro:property name="camera_resx" value="640"/>
     <xacro:property name="camera_resy" value="480"/>
@@ -31,5 +31,5 @@
             <parent link="camera_${side}_link"/>
             <child link="camera_${side}_gazebo_link"/>
-            <origin xyz="0 0 0" rpy="0 0 0"/>
+            <origin xyz="1 1 1" rpy="0 0 0"/>
             <!-- TODO: This rotation is wrong. -->
             <axis xyz="0 0 0"/>
@@ -39,5 +39,5 @@
             <xacro:weightless/>
         </link>
-        <gazebo>
+        <gazebo reference="camera_${side}_gazebo_link">
             <sensor:camera name="camera_${side}_sensor">
                 <imageSize>${camera_resx} ${camera_resy}</imageSize>
@@ -56,9 +56,4 @@
                     <Cx>${(camera_resx+1)/2}</Cx>
                     <Cy>${(camera_resy+1)/2}</Cy>
-                    <distortion_k1>0.00000001</distortion_k1>
-                    <distortion_k2>0.00000001</distortion_k2>
-                    <distortion_k3>0.00000001</distortion_k3>
-                    <distortion_t1>0.00000001</distortion_t1>
-                    <distortion_t2>0.00000001</distortion_t2>
                     <interface:camera name="camera_${side}_iface" />
                 </controller:gazebo_ros_camera>

Commit message: fixed stuff

File: navi_model/urdf/cameras.urdf.xacro (robot description, xacro)
@@ -31,5 +31,5 @@
             <parent link="camera_${side}_link"/>
             <child link="camera_${side}_gazebo_link"/>
-            <origin xyz="1 1 1" rpy="0 0 0"/>
+            <origin xyz="0 0 0" rpy="0 0 0"/>
             <!-- TODO: This rotation is wrong. -->
             <axis xyz="0 0 0"/>

File: navi_model/urdf/gps.urdf.xacro (robot description, xacro)
@@ -27,5 +27,5 @@
                 <updateRate>${gps_rate}</updateRate>
                 <bodyName>base_link</bodyName>
-                <topicName>/gps</topicName>
+                <topicName>ground_truth</topicName>
                 <gaussianNoise>${gps_sigma}</gaussianNoise>
                 <frameName>/map</frameName>

File: navi_model/urdf/laser.urdf.xacro (robot description, xacro)
@@ -37,5 +37,5 @@
                     <alwaysOn>true</alwaysOn>
                     <updateRate>20</updateRate>
-                    <topicName>/laser</topicName>
+                    <topicName>laser</topicName>
                     <frameName>/laser_link</frameName>
                     <interface:laser name="laser_iface"/>

File: navi_model/urdf/navi.urdf.xacro (robot description, xacro)
@@ -24,5 +24,4 @@
     <include filename="$(find navi_model)/urdf/wheels.urdf.xacro"/>
     <include filename="$(find navi_model)/urdf/caster.urdf.xacro"/>
-    <include filename="$(find navi_model)/urdf/sensors.urdf.xacro"/>
     <include filename="$(find navi_model)/urdf/cameras.urdf.xacro"/>
     <include filename="$(find navi_model)/urdf/laser.urdf.xacro"/>

File: navi_model/urdf/navi_robot.urdf.xacro (robot description, xacro)
@@ -47,3 +47,18 @@
         <xacro:weightless/>
     </link>
+    <gazebo>
+        <controller:diffdrive_plugin name="differential_drive_controller" plugin="libdiffdrive_plugin.so">
+            <alwaysOn>true</alwaysOn>
+            <update>100</update>
+            <updateRate>100.0</updateRate>
+            <torque>1000</torque>
+            <wheelSeparation>${wheel_offset*2}</wheelSeparation>
+            <wheelDiameter>${wheel_radius*2}</wheelDiameter>
+            <robotNamespace></robotNamespace>
+            <topicName>drive/cmd_vel</topicName>
+            <leftJoint>wheel_left_joint</leftJoint>
+            <rightJoint>wheel_right_joint</rightJoint>
+            <interface:position name="drive_iface"/>
+        </controller:diffdrive_plugin>
+    </gazebo>
 </robot>

Commit message: commented out all of the Gazebo sensors

File: navi_model/urdf/cameras.urdf.xacro (robot description, xacro)
@@ -39,4 +39,5 @@
             <xacro:weightless/>
         </link>
+        <!--
         <gazebo reference="camera_${side}_gazebo_link">
             <sensor:camera name="camera_${side}_sensor">
@@ -60,4 +61,5 @@
             </sensor:camera>
         </gazebo>
+        -->
     </xacro:macro>
 </robot>

File: navi_model/urdf/laser.urdf.xacro (robot description, xacro)
@@ -20,4 +20,5 @@
             <xacro:weightless/>
         </link>
+        <!--
         <gazebo reference="laser_link">
             <sensor:ray name="laser">
@@ -43,4 +44,5 @@
             </sensor:ray>
         </gazebo>
+        -->
     </xacro:macro>
 </robot>

File: navi_model/urdf/navi.urdf.xacro (robot description, xacro)
@@ -8,6 +8,8 @@
        xmlns:xacro="http://ros.org/wiki/xacro"
        name="navi">
+    <xacro:property name="EPS" value="0.000001"/>
     <xacro:property name="PI" value="3.1415926535897931"/>
-    <xacro:property name="EPS" value="0.000001"/>
+    <xacro:property name="robot_weight" value="90.0"/>
+    <xacro:property name="wheel_radius" value="0.127"/>
     <xacro:macro name="weightless">
         <inertial>
@@ -18,6 +20,4 @@
         </inertial>
     </xacro:macro>
-    <xacro:property name="gps_noise" value="0.005"/>
-    <xacro:property name="encoders_noise" value="0.100"/>
     <include filename="$(find navi_model)/urdf/materials.urdf.xacro"/>
     <include filename="$(find navi_model)/urdf/navi_robot.urdf.xacro"/>

File: navi_model/urdf/navi_robot.urdf.xacro (robot description, xacro)
@@ -47,4 +47,5 @@
         <xacro:weightless/>
     </link>
+    <!--
     <gazebo>
         <controller:diffdrive_plugin name="differential_drive_controller" plugin="libdiffdrive_plugin.so">
@@ -72,3 +73,4 @@
         <canonicalBody>base_footprint</canonicalBody>
     </gazebo>
+    -->
 </robot>

File: navi_model/urdf/wheels.urdf.xacro (robot description, xacro)
@@ -45,4 +45,5 @@
             <mechanicalReduction>1.0</mechanicalReduction>
         </transmission>
+        <!--
         <gazebo reference="wheel_${side}_link">
             <material>Gazebo/Red</material>
@@ -52,4 +53,5 @@
             <kd value="1.0"/>
         </gazebo>
+        -->
     </xacro:macro>
 </robot>

Commit message: added wheels, again.

File: navi_model/urdf/cameras.urdf.xacro (robot description, xacro)
@@ -7,9 +7,15 @@
        xmlns:sensor="http://playerstage.sourceforge.net/gazebo/xmlschema/#sensor"
        xmlns:xacro="http://ros.org/wiki/xacro">
+    <xacro:property name="camera_x" value="-0.09717"/>
+    <xacro:property name="camera_y" value="0.24582"/>
+    <xacro:property name="camera_z" value="0.75734"/>
+    <xacro:property name="camera_roll"  value="0"/>
+    <xacro:property name="camera_pitch" value="0.177150919"/>
+    <xacro:property name="camera_yaw"   value="0.174532925"/>
     <xacro:property name="image_width"  value="640"/>
     <xacro:property name="image_height" value="480"/>
-    <xacro:property name="hfov" value="80"/>
-    <xacro:property name="fps" value="10"/>
-    <xacro:property name="focal_length" value="320"/>
+    <xacro:property name="camera_hfov" value="80"/>
+    <xacro:property name="camera_fps" value="10"/>
+    <xacro:property name="camera_focus" value="320"/>
     <xacro:macro name="camera" params="side sign">
         <xacro:frame parent="base_link" child="camera_${side}"
@@ -20,5 +26,5 @@
             <imageSize>${image_width} ${image_height}</imageSize>
             <imageFormat>R8G8B8</imageFormat>
-            <hfov>${hfov}</hfov>
+            <hfov>${camera_hfov}</hfov>
             <nearClip>0.1</nearClip>
             <farClip>100</farClip>
@@ -26,5 +32,5 @@
             <controller:gazebo_ros_depth_camera name="camera_{$side}_controller" plugin="libgazebo_ros_depth_camera.so">
               <alwaysOn>true</alwaysOn>
-              <updateRate>25.0</updateRate>
+              <updateRate>${camera_fps}</updateRate>
               <cameraName>camera_${side}</cameraName>
               <imageTopicName>/${side}/image_raw</imageTopicName>
@@ -37,5 +43,5 @@
               <!-- image_width / (2*tan(hfov_radian /2)) -->
               <!-- 320 for wide and 772.55 for narrow stereo camera -->
-              <focalLength>${focal_length}</focalLength>
+              <focalLength>${camera_focus}</focalLength>
               <distortionK1>0.0</distortionK1>
               <distortionK2>0.0</distortionK2>

File: navi_model/urdf/chassis.urdf.xacro (robot description, xacro)
@@ -14,5 +14,5 @@
             <parent link="base_footprint"/>
             <child link="base_link"/>
-            <origin xyz="0 0 ${robot_clearance + wheel_radius}"/>
+            <origin xyz="0 0 ${wheel_radius}"/>
         </joint>
         <link name="base_link">
@@ -24,10 +24,12 @@
             </inertial>
             <visual>
-                <origin xyz="0 0.52 0.07" rpy="${PI/2} 0 0"/>
+                <origin xyz="0 0 ${2*wheel_radius}" rpy="0 0 0"/>
                 <geometry>
-                    <mesh filename="package://navi_model/meshes/frame.stl" scale="0.001 0.001 0.001"/>
+                    <box size="0.9 0.8 0.3"/>
+                    <!--<mesh filename="package://navi_model/meshes/frame.stl" scale="0.001 0.001 0.001"/>-->
                 </geometry>
             </visual>
             <collision>
+                <origin xyz="0 0 ${4*wheel_radius}" rpy="0 0 0"/>
                 <geometry>
                     <box size="0.9 0.8 0.3"/>

File: navi_model/urdf/gazebo.urdf.xacro (robot description, xacro)
@@ -16,5 +16,5 @@
                 <rightJoint>wheel_right_joint</rightJoint>
                 <wheelSeparation>${wheel_separation}</wheelSeparation>
-                <wheelDiameter>${wheel_radius*2}</wheelDiameter>
+                <wheelDiameter>${2*wheel_radius}</wheelDiameter>
                 <robotNamespace>/</robotNamespace>
                 <baseFrame>base_footprint</baseFrame>

File: navi_model/urdf/navi.urdf.xacro (robot description, xacro)
@@ -11,4 +11,5 @@
     <xacro:property name="PI" value="3.1415926535897931"/>
     <xacro:property name="robot_weight" value="90.0"/>
+    <!-- Wheels -->
     <xacro:property name="wheel_radius" value="0.127"/>
     <xacro:property name="wheel_thickness" value="0.0762"/>
@@ -16,5 +17,4 @@
     <xacro:property name="wheel_mass" value="3.175"/>
     <xacro:property name="wheel_torque" value="10"/>
-    <xacro:property name="robot_clearance" value="0.3937"/>
     <xacro:property name="caster_radius" value="0.1143"/>
     <xacro:property name="caster_thickness" value="0.0508"/>
@@ -27,10 +27,4 @@
     <xacro:property name="gps_offset" value="-0.18941 0 0.76387"/>
     <xacro:property name="laser_offset" value="0.02927 0 0.46714"/>
-    <xacro:property name="camera_x" value="-0.09717"/>
-    <xacro:property name="camera_y" value="0.24582"/>
-    <xacro:property name="camera_z" value="0.75734"/>
-    <xacro:property name="camera_roll"  value="0"/>
-    <xacro:property name="camera_pitch" value="0.177150919"/>
-    <xacro:property name="camera_yaw"   value="0.174532925"/>
     <xacro:macro name="weightless">
         <inertial>
@@ -56,10 +50,14 @@
     <xacro:wheel sign="+1" side="left"/>
     <xacro:wheel sign="-1" side="right"/>
+    <!--
     <xacro:caster/>
+    -->
     <xacro:camera sign="+1" side="left"/>
     <xacro:camera sign="-1" side="right"/>
     <xacro:frame parent="base_link" child="gps" xyz="${gps_offset}" rpy="0 0 0"/>
     <xacro:frame parent="base_link" child="laser" xyz="${laser_offset}" rpy="0 0 0"/>
+    <!--
     <xacro:gazebo_drive/>
     <xacro:gazebo_localization/>
+    -->
 </robot>

File: navi_model/urdf/wheels.urdf.xacro (robot description, xacro)
@@ -11,5 +11,5 @@
             <parent link="base_link"/>
             <child link="wheel_${side}_link"/>
-            <origin xyz="0 ${sign*wheel_separation/2} ${-robot_clearance}" rpy="${PI/2} 0 0"/>
+            <origin xyz="0 ${0.5*sign*wheel_separation} 0" rpy="${PI/2} 0 0"/>
             <axis xyz="0 0 1"/>
         </joint>
@@ -52,5 +52,4 @@
             </inertial>
         </link>
-        <!-- TODO: Why can't I make this continuous? -->
         <joint name="caster_joint" type="fixed">
             <parent link="caster_pivot_link"/>

Commit message: full CV stack running

File: navi_model/urdf/cameras.urdf.xacro (robot description, xacro)
@@ -11,5 +11,5 @@
     <xacro:property name="camera_z" value="0.75734"/>
     <xacro:property name="camera_roll"  value="0"/>
-    <xacro:property name="camera_pitch" value="0.177150919"/>
+    <xacro:property name="camera_pitch" value="0.593411946"/>
     <xacro:property name="camera_yaw"   value="0.174532925"/>
     <xacro:property name="image_width"  value="640"/>
