Commit message: added wheels

File: navi_model/object.urdf (robot description, URDF)
Before this commit: robot simple_box, 1 links, 0 joints
Links:
- removed link my_box
- added link base_link, mass 1.0; collision box size=0.9 0.8 0.3; visual box size=0.9 0.8 0.3
- added link wheel_left_link, mass 1.0; collision box size=0.2 0.2 0.2; visual box size=0.2 0.2 0.2
- added link wheel_right_link, mass 1.0; collision box size=0.2 0.2 0.2; visual box size=0.2 0.2 0.2
Joints:
- added joint wheel_left_joint: type fixed, parent base_link, child wheel_left_link, origin xyz=0 1 0
- added joint wheel_right_joint: type fixed, parent base_link, child wheel_right_link, origin xyz=0 -1 0

Commit message: added a block caster

File: navi_model/object.urdf (robot description, URDF)
Before this commit: robot simple_box, 3 links, 2 joints
Links:
- added link caster_link, mass 1.0; collision box size=0.2 0.2 0.2; visual box size=0.2 0.2 0.2
Joints:
- added joint caster_joint: type fixed, parent base_link, child caster_link, origin xyz=-1 0 0

Commit message: closer...

File: navi_model/object.urdf (robot description, URDF)
Before this commit: robot simple_box, 4 links, 3 joints
Links:
- link caster_link: geometry collision cylinder length=0.05 radius=0.127; visual cylinder length=0.05 radius=0.127
- link wheel_left_link: geometry collision cylinder length=0.05 radius=0.127; visual cylinder length=0.05 radius=0.127
- link wheel_right_link: geometry collision cylinder length=0.05 radius=0.127; visual cylinder length=0.05 radius=0.127
Joints:
- joint caster_joint: origin xyz=-1 0 0 -> xyz=-1 0 0 rpy=1.57 0 0
- joint wheel_left_joint: origin xyz=0 1 0 -> xyz=0 1 0 rpy=1.57 0 0
- joint wheel_right_joint: origin xyz=0 -1 0 -> xyz=0 -1 0 rpy=1.57 0 0
